File: analog-via.kicad_pcb (KiCad board)
At the start: 2 copper layers, 213.5 x 128.5 mm, 708 parts, among them IC1 SSI2164, IC2 SSI2164, J1 2164_CV, J10 2164_IN, J11 SLEW_CV, J12 2164_CTL, J13 2164_OUT, J14 INTEGRATOR_IN, J15 COMP_CTL_A, J16 HIGH_COMP, J17 LOW_COMP, J18 INTEGRATOR, J19 OUTPUT, J2 5VREF, J20 COMP_CTL_B, J21 INV_SLOPE, J22 SLOPE, J23 POWER, J24 SYNC, J25 TRIGGER, J26 SYNC, J27 RISE, J28 FALL, J29 INA, J3 EXPO_IN, J30 INB, J31 OUTPUT, J32 DIRECTION, J33 EOC, J34 SLOPE, J35 CLK/2, J36 FALL_SUM, J37 RISE_SUM, J39 2.5VREF, J4 FF_TRIGGER, J40 SLOPE_FREQ_MOD, J41 INA, J42 INB, J43 Conn_01x06, J44 EXTRA_SW_B, J45 EXTRA_SW_C, J46 LOGIC_S1, J47 LOGIC_S2, J48 LOGIC_S3, J49 Conn_01x03, J5 ONESHOT_OR_RETRIG, J50 1V/OCT, J6 TRIGGER, J7 EOC, J8 HOLD_REF, J9 INPUT, Q1 MMBFJ112, Q2 PNP, U1 74HC74, U11 OPA1678, U12 LM311, U13 LM311, U14 OPA1678, U15 OPA1678, U16 TMUX4053PWR, U18 AMS1117-5.0, U19 TMUX4053PWR, U2 LM4040DBZ-5, U3 TMUX4053PWR, U4 OPA1678, U5 LM339, U7 OPA1678, U9 OPA1679

Commit message: rotated op amp packages and corrected power supply issues, ratsnest still needs corrections
Parts:
- D2: value D_Schottky -> 1N5819
- R1: value 840 -> 845
- R26: value 47.5k -> 47k
- R6: value 339 -> 340
- moved R59 1.54 mm to (162.9, 66.9), turned to 0 degrees
- moved R55 1.44 mm to (161.7, 77.8), turned to 0 degrees
- turned U11 to -90 degrees
- turned U14 to -90 degrees
- turned U15 to -90 degrees
- turned U4 to -90 degrees
- turned U7 to -90 degrees
- turned U9 to -90 degrees
Connections:
- R20 pad 2: Net-(U4A-+) -> Net-(U4B-+)
- R21 pad 1: Net-(U4A--) -> Net-(U4B--)
- R51 pad 2: Net-(U11A--) -> Net-(U11B--)
- R52 pad 1: Net-(U11A--) -> Net-(U11B--)
- R55 pad 1: Net-(U11A--) -> Net-(U11B--)
- R57 pad 2: Net-(U11B--) -> Net-(U11A--)
- R59 pad 1: Net-(U11B--) -> Net-(U11A--)
- R69 pad 2: Net-(U15A--) -> Net-(U15B--)
- R71 pad 1: Net-(U15A--) -> Net-(U15B--)
- U11 pad 1: INV_SLOPE -> SLOPE
- U11 pad 4: +12V -> -12V
- U11 pad 7: SLOPE -> INV_SLOPE
- U11 pad 8: -12V -> +12V
- U14 pad 1: SLOPE_SW_RISE -> SLOPE_SW_FALL
- U14 pad 2: Net-(J36-Pin_1) -> Net-(J37-Pin_1)
- U14 pad 4: +12V -> -12V
- U14 pad 6: Net-(J37-Pin_1) -> Net-(J36-Pin_1)
- U14 pad 7: SLOPE_SW_FALL -> SLOPE_SW_RISE
- U14 pad 8: -12V -> +12V
- U15 pad 1: SLOPE_FREQ_MOD -> Net-(JP6-A)
- U15 pad 2: Net-(U15A--) -> Net-(JP6-B)
- U15 pad 3: GND -> Net-(JP5-B)
- U15 pad 4: +12V -> -12V
- U15 pad 5: Net-(JP5-B) -> GND
- U15 pad 6: Net-(JP6-B) -> Net-(U15B--)
- U15 pad 7: Net-(JP6-A) -> SLOPE_FREQ_MOD
- U15 pad 8: -12V -> +12V
- U4 pad 1: A0 -> Net-(JP2-A)
- U4 pad 2: Net-(U4A--) -> Net-(JP2-B)
- U4 pad 3: Net-(U4A-+) -> Net-(JP1-B)
- U4 pad 4: +12V -> -12V
- U4 pad 5: Net-(JP1-B) -> Net-(U4B-+)
- U4 pad 6: Net-(JP2-B) -> Net-(U4B--)
- U4 pad 7: Net-(JP2-A) -> A0
- U4 pad 8: -12V -> +12V
- U7 pad 1: Net-(J18-Pin_2) -> Net-(IC1A-CTRL)
- U7 pad 2: B -> Net-(IC1C-OUT)
- U7 pad 4: +12V -> -12V
- U7 pad 6: Net-(IC1C-OUT) -> B
- U7 pad 7: Net-(IC1A-CTRL) -> Net-(J18-Pin_2)
- U7 pad 8: -12V -> +12V
- U9 pad 1: Net-(C8-Pad2) -> Net-(JP4-A)
- U9 pad 11: +12V -> -12V
- U9 pad 12: Net-(JP3-B) -> GND
- U9 pad 13: Net-(JP4-B) -> Net-(IC2A-OUT)
- U9 pad 14: Net-(JP4-A) -> Net-(C8-Pad2)
- U9 pad 2: Net-(IC2A-OUT) -> Net-(JP4-B)
- U9 pad 3: GND -> Net-(JP3-B)
- U9 pad 4: -12V -> +12V
- U9 pad 6: Net-(IC2C-OUT) -> Net-(IC2B-OUT)
- U9 pad 7: Net-(C16-Pad2) -> OUTPUT
- U9 pad 8: OUTPUT -> Net-(C16-Pad2)
- U9 pad 9: Net-(IC2B-OUT) -> Net-(IC2C-OUT)
Routing:
- net GND: track 233.4 -> 220.1 mm, vias 100 -> 93
- net Net-(U15B--): track 0.00 -> 8.65 mm
- net Net-(U15A--): track 8.65 -> 0.00 mm
- net Net-(U11B--): track 7.23 -> 15.2 mm
- net Net-(U11A--): track 15.2 -> 7.23 mm
- net Net-(U4B-+): track 0.00 -> 6.03 mm
- net Net-(U4A-+): track 6.03 -> 0.00 mm
- net SLOPE_SW_RISE: track 37.7 -> 41.0 mm, vias 2 -> 4
- net SLOPE_FREQ_MOD: track 91.3 -> 94.5 mm, vias 1 -> 3
- net Net-(U4B--): track 0.00 -> 2.98 mm
- net Net-(U4A--): track 2.98 -> 0.00 mm
- net Net-(J18-Pin_2): track 76.5 -> 78.6 mm, vias 4 -> 5
- net INV_SLOPE: track 84.6 -> 86.6 mm
- net Net-(IC1A-CTRL): track 58.2 -> 60.1 mm, vias 2 -> 3
- net SLOPE_SW_FALL: track 38.7 -> 40.5 mm, vias 2 -> 3
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