File: analog-via.kicad_pcb (KiCad board)
At the start: 2 copper layers, 213.5 x 128.5 mm, 708 parts, among them IC1 SSI2164, IC2 SSI2164, J1 2164_CV, J10 2164_IN, J11 SLEW_CV, J12 2164_CTL, J13 2164_OUT, J14 INTEGRATOR_IN, J15 COMP_CTL_A, J16 HIGH_COMP, J17 LOW_COMP, J18 INTEGRATOR, J19 OUTPUT, J2 5VREF, J20 COMP_CTL_B, J21 INV_SLOPE, J22 SLOPE, J23 POWER, J24 SYNC, J25 TRIGGER, J26 SYNC, J27 RISE, J28 FALL, J29 INA, J3 EXPO_IN, J30 INB, J31 OUTPUT, J32 DIRECTION, J33 EOC, J34 SLOPE, J35 CLK/2, J36 FALL_SUM, J37 RISE_SUM, J39 2.5VREF, J4 FF_TRIGGER, J40 SLOPE_FREQ_MOD, J41 INA, J42 INB, J43 Conn_01x06, J44 EXTRA_SW_B, J45 EXTRA_SW_C, J46 LOGIC_S1, J47 LOGIC_S2, J48 LOGIC_S3, J49 Conn_01x03, J5 ONESHOT_OR_RETRIG, J50 1V/OCT, J6 TRIGGER, J7 EOC, J8 HOLD_REF, J9 INPUT, Q1 MMBFJ112, Q2 PNP, U1 74HC74, U11 OPA1678, U12 LM311, U13 LM311, U14 OPA1678, U15 OPA1678, U16 TMUX4053PWR, U18 AMS1117-5.0, U19 TMUX4053PWR, U2 LM4040DBZ-5, U3 TMUX4053PWR, U4 OPA1678, U5 LM339, U7 OPA1678, U9 OPA1679

Commit message: routing
Parts:
- removed C14, C29, C36: 100n, Capacitor_SMD:C_0805_2012Metric
- removed D1: 1N5819, Diode_SMD:D_SOD-123
- removed D2: D_Schottky, Diode_SMD:D_SOD-123
- removed J33: EOC, Connector_Audio:Jack_3.5mm_QingPu_WQP-PJ398SM_Vertical_CircularHoles
- removed J34: SLOPE, Connector_Audio:Jack_3.5mm_QingPu_WQP-PJ398SM_Vertical_CircularHoles
- removed J35: CLK/2, Connector_Audio:Jack_3.5mm_QingPu_WQP-PJ398SM_Vertical_CircularHoles
- removed J43: Conn_01x06, Connector_PinHeader_2.54mm:PinHeader_1x06_P2.54mm_Vertical
- removed J45: EXTRA_SW_C, Connector_PinHeader_2.54mm:PinHeader_1x01_P2.54mm_Vertical
- removed J46: LOGIC_S1, Connector_PinHeader_2.54mm:PinHeader_1x01_P2.54mm_Vertical
- removed J47: LOGIC_S2, Connector_PinHeader_2.54mm:PinHeader_1x01_P2.54mm_Vertical
- removed J48: LOGIC_S3, Connector_PinHeader_2.54mm:PinHeader_1x01_P2.54mm_Vertical
- removed J49: Conn_01x03, Connector_PinHeader_2.54mm:PinHeader_1x03_P2.54mm_Vertical
- removed Q1: MMBFJ112, Package_TO_SOT_SMD:SOT-23
- removed Q2: PNP, Package_TO_SOT_SMD:SOT-23-3
- removed R12, R13, R14, R15, R16, R66, R67, R68: 100k, Resistor_SMD:R_0805_2012Metric
- removed R17, R22, R23, R45, R48, R65, R70: 10k, Resistor_SMD:R_0805_2012Metric
- removed R27, R28, R29: 33k, Resistor_SMD:R_0805_2012Metric
- removed R50, R60, R74, R75: 1k, Resistor_SMD:R_0805_2012Metric
- removed R72, R73: 1K, Resistor_SMD:R_0805_2012Metric
- removed REF**, REF**1, REF**10, REF**100 (x11), REF**101 (x17), REF**102 (x2), REF**103 (x2), REF**104, REF**105, REF**106, REF**107, REF**108 (x8), REF**109 (x11), REF**11, REF**110 (x11), REF**111 (x17), REF**112 (x2), REF**113 (x2), REF**114, REF**115, REF**116, REF**117, REF**118 (x10), REF**119 (x12), REF**12, REF**120 (x14), REF**121 (x22), REF**125 (x2), REF**126 (x2), REF**127 (x2), REF**128 (x6), REF**129 (x6), REF**13, REF**130 (x6), REF**131 (x8), REF**14, REF**15, REF**2, REF**20 (x8), REF**21 (x11), REF**22 (x11), REF**23 (x17), REF**24 (x2), REF**25 (x2), REF**3, REF**30, REF**31, REF**32, REF**33, REF**34 (x8), REF**35 (x11), REF**4, REF**40 (x11), REF**41 (x17), REF**42 (x2), REF**43 (x2), REF**44, REF**45, REF**5, REF**50, REF**51, REF**52 (x8), REF**53 (x11), REF**54 (x11), REF**55 (x17), REF**6 (x3), REF**60 (x2), REF**61 (x2), REF**62, REF**63, REF**64, REF**65, REF**7 (x3), REF**70 (x8), REF**71 (x11), REF**72 (x11), REF**73 (x17), REF**74 (x2), REF**75 (x2), REF**8 (x3), REF**80, REF**81, REF**82, REF**83, REF**84 (x8), REF**85 (x11), REF**9 (x4), REF**90 (x11), REF**91 (x17), REF**92 (x2), REF**93 (x2), REF**94, REF**95, REF**96, REF**97, REF**98 (x8), REF**99 (x11): PinHeader_1x01_P2.54mm_Vertical, Connector_PinHeader_2.54mm:PinHeader_1x01_P2.54mm_Vertical
- removed REF** (x4): MountingHole_3.2mm_M3_Pad, MountingHole:MountingHole_3.2mm_M3_Pad
- removed U15: OPA1678, Package_SO:SOIC-8_3.9x4.9mm_P1.27mm
- removed U5: LM339, Package_SO:SOIC-14_3.9x8.7mm_P1.27mm
- added C46: 100n, Capacitor_SMD:C_0805_2012Metric, F.Cu at (252.0, 154.1)
- added C47: 100p, Capacitor_SMD:C_0805_2012Metric, F.Cu at (-53.0, 70.9)
- added C50: 1.2n, Capacitor_SMD:C_0805_2012Metric, F.Cu at (-32.5, 10.3)
- added C51: 1.2n, Capacitor_SMD:C_0805_2012Metric, F.Cu at (247.1, 157.1)
- added C52: 1200p, Capacitor_SMD:C_0805_2012Metric, F.Cu at (113.9, 90.8)
- added C53: 1uF, Capacitor_SMD:C_0805_2012Metric, F.Cu at (93.8, 38.5)
- added C54: 100n, Capacitor_SMD:C_0805_2012Metric, F.Cu at (91.5, 194.7)
- added C55: 100nF, Capacitor_SMD:C_0805_2012Metric, F.Cu at (30.6, 184.2)
- added C58: 100n, Capacitor_SMD:C_0805_2012Metric, F.Cu at (-64.8, 74.9)
- added C59: 100n, Capacitor_SMD:C_0805_2012Metric, F.Cu at (-67.4, 63.5)
- added C60: 100n, Capacitor_SMD:C_0805_2012Metric, F.Cu at (50.2, 166.2)
- added C61: 100n, Capacitor_SMD:C_0805_2012Metric, F.Cu at (-45.3, 65.1)
- added C62: 100n, Capacitor_SMD:C_0805_2012Metric, F.Cu at (-29.5, 12.3)
- added D3: 1N5819, Diode_SMD:D_SOD-123, F.Cu at (-53.7, 67.1)
- added D4: 1n4148, Diode_SMD:D_SOD-123, F.Cu at (18.7, 192.0)
- added D5: LED, LED_SMD:LED_0805_2012Metric, F.Cu at (50.7, 194.2)
- added D6: LED, LED_SMD:LED_0805_2012Metric, F.Cu at (50.7, 190.6)
- added D7: LED, LED_SMD:LED_0805_2012Metric, F.Cu at (50.6, 186.8)
- added D8: LED, LED_SMD:LED_0805_2012Metric, F.Cu at (50.6, 182.8)
- added J38: Conn_02x02_Counter_Clockwise, Connector_PinHeader_2.54mm:PinHeader_2x02_P2.54mm_Vertical, F.Cu at (80.0, -18.1)
- added J60: Conn_01x02, Connector_PinHeader_2.54mm:PinHeader_1x02_P2.54mm_Vertical, F.Cu at (-25.4, 146.5)
- added J64: HOLD_REF_INV, Connector_PinHeader_2.54mm:PinHeader_1x01_P2.54mm_Vertical, F.Cu at (109.6, 80.4)
- added J65: Conn_01x02, Connector_PinHeader_2.54mm:PinHeader_1x02_P2.54mm_Vertical, F.Cu at (41.3, -15.0)
- added J67: Conn_01x01, Connector_PinHeader_2.54mm:PinHeader_1x01_P2.54mm_Vertical, F.Cu at (73.6, 179.8)
- added R100: 1k, Resistor_SMD:R_0805_2012Metric, F.Cu at (46.9, 186.8)
- added R101: 1k, Resistor_SMD:R_0805_2012Metric, F.Cu at (47.0, 182.8)
- added R102: 100k, Resistor_SMD:R_0805_2012Metric, F.Cu at (-53.9, 73.9)
- added R103: 10k, Resistor_SMD:R_0805_2012Metric, F.Cu at (-67.2, 77.0)
- added R104: 100k, Resistor_SMD:R_0805_2012Metric, F.Cu at (-64.1, 77.8)
- added R105: 1M, Resistor_SMD:R_0805_2012Metric, F.Cu at (-70.5, 69.4)
- added R106: 4.7k, Resistor_SMD:R_0805_2012Metric, F.Cu at (-69.7, 63.5)
- added R107: 100k, Resistor_SMD:R_0805_2012Metric, F.Cu at (-71.4, 72.6)
- added R108: 1M, Resistor_SMD:R_0805_2012Metric, F.Cu at (28.4, 123.0)
- added R109: 1, Resistor_SMD:R_0805_2012Metric, F.Cu at (33.5, 131.2)
- added R110: 100k, Resistor_SMD:R_0805_2012Metric, F.Cu at (-49.1, 65.1)
- added R82: 200k, Resistor_SMD:R_0805_2012Metric, F.Cu at (-37.2, 7.90)
- added R83: 10k, Resistor_SMD:R_0805_2012Metric, F.Cu at (-63.1, 63.3)
- added R84: 100k, Resistor_SMD:R_0805_2012Metric, F.Cu at (-64.8, 59.7)
- added R85: 200k, Resistor_SMD:R_0805_2012Metric, F.Cu at (-32.5, 6.70)
- added R86: 1M, Resistor_SMD:R_0805_2012Metric, F.Cu at (-59.1, 69.1)
- added R87: 4.7k, Resistor_SMD:R_0805_2012Metric, F.Cu at (-59.1, 72.7)
- added R90: 33k, Resistor_SMD:R_0805_2012Metric, F.Cu at (-22.4, 7.40)
- added R91: 220, Resistor_SMD:R_0805_2012Metric, F.Cu at (116.2, 90.8)
- added R92: 845, Resistor_SMD:R_0805_2012Metric, F.Cu at (91.5, 25.4)
- added R93: 150k, Resistor_SMD:R_0805_2012Metric, F.Cu at (18.7, 187.3)
- added R94: 100k, Resistor_SMD:R_0805_2012Metric, F.Cu at (22.1, 185.0)
- added R95: 300k, Resistor_SMD:R_0805_2012Metric, F.Cu at (22.6, 191.2)
- added R96: 300k, Resistor_SMD:R_0805_2012Metric, F.Cu at (22.6, 193.4)
- added R97: 600k, Resistor_SMD:R_0805_2012Metric, F.Cu at (22.6, 188.8)
- added R98: 1k, Resistor_SMD:R_0805_2012Metric, F.Cu at (46.9, 194.2)
- added R99: 1k, Resistor_SMD:R_0805_2012Metric, F.Cu at (46.9, 190.6)
- added RV4: 100k, Potentiometer_THT:Potentiometer_TT_P0915N, F.Cu at (23.2, 179.3)
- added U10: 74LS08, Package_SO:SOIC-14_3.9x8.7mm_P1.27mm, F.Cu at (93.5, 179.9)
- added U17: LM319, Package_SO:SOIC-14_3.9x8.7mm_P1.27mm, F.Cu at (-64.8, 69.3)
- added U22: 74AHC1G32, Package_TO_SOT_SMD:SOT-23-5, F.Cu at (82.8, 189.0)
- added U30: 74AHC1G86, Package_TO_SOT_SMD:SOT-353_SC-70-5, F.Cu at (54.4, 165.8)
- added U32: LF398_SOIC14, Package_SO:SOIC-14_3.9x8.7mm_P1.27mm, F.Cu at (40.0, -22.0)
- added U33: OPA1678, Package_SO:SOIC-8_3.9x4.9mm_P1.27mm, F.Cu at (-27.5, 8.34)
- added U35: OPA1678, Package_SO:SOIC-8_3.9x4.9mm_P1.27mm, F.Cu at (248.1, 152.1)
- added U37: TL431DBZ, Package_TO_SOT_SMD:SOT-23, F.Cu at (109.7, 85.4)
- added U39: 74HC14, Package_SO:SOIC-14_3.9x8.7mm_P1.27mm, F.Cu at (44.4, 164.2)
- added U40: 74HC14, Package_SO:SOIC-14_3.9x8.7mm_P1.27mm, F.Cu at (-47.2, 70.9)
- added U42: 74HC237, Package_SO:SOIC-16_4.55x10.3mm_P1.27mm, F.Cu at (38.7, 189.2)
- added U6: TMUX4053, Package_SO:TSSOP-16_4.4x5mm_P0.65mm, F.Cu at (62.7, 165.9)
- added U8: LM3900, Package_SO:SOIC-14_3.9x8.7mm_P1.27mm, F.Cu at (28.6, 189.9)
- C13: value 1.2n -> 100n
- C27, C28: value 100p -> 100n
- J10: value 2164_IN -> TRIGGER
- J12: value 2164_CTL -> Conn_02x04_Odd_Even; footprint Connector_PinHeader_2.54mm:PinHeader_1x01_P2.54mm_Vertical -> Connector_PinHeader_2.54mm:PinHeader_2x04_P2.54mm_Vertical
- J13: value 2164_OUT -> Conn_01x04; footprint Connector_PinHeader_2.54mm:PinHeader_1x01_P2.54mm_Vertical -> Connector_PinHeader_2.54mm:PinHeader_1x04_P2.54mm_Vertical
- J14: value INTEGRATOR_IN -> INB; footprint Connector_PinHeader_2.54mm:PinHeader_1x01_P2.54mm_Vertical -> Connector_Audio:Jack_3.5mm_QingPu_WQP-PJ398SM_Vertical_CircularHoles
- J16: value HIGH_COMP -> LOW_COMP
- J17: value LOW_COMP -> HIGH_COMP
- J18: value INTEGRATOR -> Conn_01x02_Pin
- J24: value SYNC -> TRIGGER; footprint Connector_PinHeader_2.54mm:PinHeader_1x01_P2.54mm_Vertical -> Connector_Audio:Jack_3.5mm_QingPu_WQP-PJ398SM_Vertical_CircularHoles
- J25: value TRIGGER -> SYNC
- J26: value SYNC -> RISE
- J27: value RISE -> FALL
- J28: value FALL -> INA
- J29: value INA -> CLK/2
- J30: value INB -> Conn_01x04; footprint Connector_Audio:Jack_3.5mm_QingPu_WQP-PJ398SM_Vertical_CircularHoles -> Connector_PinHeader_2.54mm:PinHeader_1x04_P2.54mm_Vertical
- J31: value OUTPUT -> Conn_01x04; footprint Connector_Audio:Jack_3.5mm_QingPu_WQP-PJ398SM_Vertical_CircularHoles -> Connector_PinHeader_2.54mm:PinHeader_1x04_P2.54mm_Vertical
- J32: value DIRECTION -> Conn_02x04_Odd_Even; footprint Connector_Audio:Jack_3.5mm_QingPu_WQP-PJ398SM_Vertical_CircularHoles -> Connector_PinHeader_2.54mm:PinHeader_2x04_P2.54mm_Vertical
- J39: value 2.5VREF -> Conn_01x02_Pin; footprint Connector_PinHeader_2.54mm:PinHeader_1x01_P2.54mm_Vertical -> Connector_PinHeader_2.54mm:PinHeader_1x02_P2.54mm_Vertical
- J4: value FF_TRIGGER -> FF_DIRECTION
- J44: value EXTRA_SW_B -> ~{SYNC}
- J5: value ONESHOT_OR_RETRIG -> SLOPE; footprint Connector_PinHeader_2.54mm:PinHeader_1x01_P2.54mm_Vertical -> Connector_Audio:Jack_3.5mm_QingPu_WQP-PJ398SM_Vertical_CircularHoles
- J6: value TRIGGER -> EOC; footprint Connector_PinHeader_2.54mm:PinHeader_1x01_P2.54mm_Vertical -> Connector_Audio:Jack_3.5mm_QingPu_WQP-PJ398SM_Vertical_CircularHoles
- J7: value EOC -> OUTPUT; footprint Connector_PinHeader_2.54mm:PinHeader_1x01_P2.54mm_Vertical -> Connector_Audio:Jack_3.5mm_QingPu_WQP-PJ398SM_Vertical_CircularHoles
- J9: value INPUT -> DIRECTION
- R1: value 840 -> 845
- R10, R5: value 1M -> 1k
- R11: value 100k -> 1K
- R18: value 100k 1% -> 100k
- R19: value 100k 1% -> 150k
- R2: value 10k -> 1K
- R26: value 47.5k -> 47k
- R40, R41: value 1M -> DNP
- R6: value 339 -> 340
- R69: value 100k -> 10M
- R71: value 100k -> 33k
- R8: value 10k -> 1k
- U16, U19, U3: value TMUX4053PWR -> TMUX4053
- moved J31 269.2 mm to (-41.6, 77.2), turned to 180 degrees
- moved J32 260.0 mm to (-36.5, 77.2), turned to 180 degrees
- moved J29 216.3 mm to (223.3, 121.0), turned to -90 degrees
- moved C23 207.8 mm to (247.1, 147.2), turned to 0 degrees
- moved JP5 181.1 mm to (236.9, 100.9)
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Connections:
- net FF_TRIGGER renamed FF_DIRECTION
- C1 pad 1: 5VREF -> Net-(U37-K)
- C13 pad 1: B -> +5V
- C13 pad 2: Net-(J18-Pin_2) -> GND
- C27 pad 1: Net-(D2-K) -> +5V
- C27 pad 2: Net-(C27-Pad2) -> GND
- C28 pad 1: GND -> +12V
- C28 pad 2: SYNC -> GND
- C3 pad 2: Net-(IC1A-CTRL) -> SLEW_CV
- C31 pad 1: -12V -> GND
- C31 pad 2: GND -> -12V
- C44 pad 1: -12V -> GND
- C44 pad 2: GND -> -12V
- IC1 pad 14: Net-(IC1D-CTRL) -> SLEW_CV
- IC1 pad 3: Net-(IC1A-CTRL) -> SLEW_CV
- IC1 pad 4: B0 -> Net-(IC1A-OUT)
- IC1 pad 6: Net-(IC1A-CTRL) -> SLEW_CV
- J10 pad 1: Net-(IC1D-IN) -> TRIGGER
- J11 pad 1: Net-(IC1A-CTRL) -> SLEW_CV
- J12 pad 1: Net-(IC1D-CTRL) -> FULL_CYCLE_MODE
- J13 pad 1: Net-(IC1D-OUT) -> +5V
- J16 pad 1: C0 -> Net-(J16-Pin_1)
- J17 pad 1: C1 -> Net-(J17-Pin_1)
- J18 pad 1: Net-(J18-Pin_1) -> GATE
- J23 pad 1: +12V -> -12V
- J23 pad 10: -12V -> +12V
- J23 pad 2: +12V -> -12V
- J23 pad 9: -12V -> +12V
- J25 pad T: TRIGGER_IN -> SYNC_IN
- J25 pad TN: GND -> unconnected-(J25-PadTN)
- J26 pad T: SYNC_IN -> RISE_CV
- J27 pad T: RISE_CV -> FALL_CV
- J28 pad T: FALL_CV -> INA
- J29 pad S: GND -> unconnected-(J29-PadS)
- J29 pad T: INA -> Net-(J29-PadT)
- J39 pad 1: 2.5VREF -> Net-(J39-Pin_1)
- J44 pad 1: Net-(J44-Pin_1) -> ~{SYNC}
- J8 pad 1: A -> HOLD_REF
- J9 pad T: Net-(J9-Pad1) -> Net-(J9-PadT)
- J9 pad TN: A -> unconnected-(J9-PadTN)
- R1 pad 1: +12V -> Net-(U37-K)
- R1 pad 2: 5VREF -> +12V
- R10 pad 1: Net-(D1-K) -> DIRECTION
- R10 pad 2: TRIGGER -> Net-(J9-PadT)
- R11 pad 1: +5V -> CLK/2
- R11 pad 2: Net-(U5C--) -> Net-(J29-PadT)
- R18 pad 1: 2.5VREF -> MODE_CV
- R18 pad 2: 5VREF -> Net-(U8A-+)
- R19 pad 1: GND -> Net-(R19-Pad1)
- R19 pad 2: 2.5VREF -> Net-(U8A-+)
- R2 pad 1: TRIGGER_IN -> SLOPE
- R2 pad 2: Net-(D1-K) -> Net-(J5-PadT)
- R20 pad 2: Net-(U4A-+) -> Net-(U4A--)
- R21 pad 2: A0 -> -5V
- R30 pad 1: Net-(J9-Pad1) -> HOLD_REF
- R33 pad 2: A0 -> -5V
- R36 pad 1: 5VREF -> +5V
- R36 pad 2: AT_TARGET -> ~{BOUNDS}
- R40 pad 1: C0 -> Net-(J16-Pin_1)
- R41 pad 1: C1 -> Net-(J17-Pin_1)
- R42 pad 2: A0 -> -5V
- R43 pad 2: A0 -> -5V
- R44 pad 1: Net-(U13-+) -> Net-(J38-Pin_1)
- R44 pad 2: 5VREF -> Net-(U13-+)
- R5 pad 1: GND -> EOC
- R5 pad 2: Net-(D1-K) -> Net-(J6-PadT)
- R51 pad 1: Net-(J18-Pin_1) -> Net-(J38-Pin_1)
- R52 pad 2: A0 -> -5V
- R58 pad 2: A0 -> -5V
- R6 pad 1: 5VREF -> Net-(U37-K)
- R63 pad 2: SLOPE_SW_RISE -> Net-(R63-Pad2)
- R64 pad 2: SLOPE_SW_FALL -> Net-(R64-Pad2)
- R69 pad 1: SLOPE_SW_OUT -> Net-(IC1D-OUT)
- R69 pad 2: Net-(U15A--) -> GND
- R71 pad 1: Net-(U15A--) -> HOLD_REF_INV
- R71 pad 2: SLOPE_FREQ_MOD -> Net-(IC1D-IN)
- R78 pad 1: LOGIC_S2 -> PENDULUM_MODE
- R79 pad 1: LOGIC_S3 -> GATE_MODE
- R8 pad 1: Net-(U5C--) -> OUTPUT
- R8 pad 2: GND -> Net-(J7-PadT)
- R80 pad 1: LOGIC_S1 -> ENV_MODE
- RV1 pad 2: Net-(IC1A-CTRL) -> SLEW_CV
- RV1 pad 3: Net-(IC1A-CTRL) -> SLEW_CV
- RV2 pad 1: GND -> -5V
- RV2 pad 3: +5V -> 5VREF
- RV3 pad 1: GND -> -5V
- RV3 pad 3: +5V -> 5VREF
- U1 pad 1: unconnected-(U1A-~{R}-Pad1) -> ACTIVATION_TRIG
- U1 pad 10: unconnected-(U1B-~{S}-Pad10) -> ~{SYNC}
- U1 pad 11: Net-(U1B-C) -> DIR_CHANGE
- U1 pad 13: SYNC -> +5V
- U1 pad 2: Net-(U1A-D) -> GND
- U1 pad 3: A_SW -> GND
- U1 pad 4: unconnected-(U1A-~{S}-Pad4) -> ~{BOUNDS}
- U1 pad 5: CLK/2 -> AT_TARGET
- U1 pad 6: Net-(U1A-D) -> unconnected-(U1A-~{Q}-Pad6)
- U11 pad 4: +12V -> -12V
- U11 pad 8: -12V -> +12V
- U12 pad 3: Net-(J18-Pin_2) -> Net-(J38-Pin_1)
- U12 pad 6: unconnected-(U12-STRB-Pad6) -> AT_TARGET
- U12 pad 7: C0 -> Net-(J16-Pin_1)
- U13 pad 3: Net-(J18-Pin_2) -> 5VREF
- U13 pad 6: unconnected-(U13-STRB-Pad6) -> AT_TARGET
- U13 pad 7: C1 -> Net-(J17-Pin_1)
- U14 pad 1: SLOPE_SW_RISE -> Net-(R63-Pad2)
- U14 pad 4: +12V -> -12V
- U14 pad 7: SLOPE_SW_FALL -> Net-(R64-Pad2)
- U14 pad 8: -12V -> +12V
- U16 pad 1: A -> 5VREF
- U16 pad 10: AT_TARGET -> INV_DIRECTION
- U16 pad 11: A_SW -> DIRECTION
- U16 pad 12: A0 -> -5V
- U16 pad 14: A -> HOLD_REF
- U16 pad 15: B -> HOLD_REF_INV
- U16 pad 2: B0 -> -5V
- U16 pad 3: C1 -> Net-(R64-Pad2)
- U16 pad 4: AT_TARGET -> SLOPE_FREQ_MOD
- U16 pad 5: C0 -> Net-(R63-Pad2)
- U16 pad 9: A_SW -> DIRECTION
- U18 pad 2: +5V -> Net-(U18-VO)
- U19 pad 1: Net-(J43-Pin_1) -> Net-(J30-Pin_3)
- U19 pad 10: Net-(J45-Pin_1) -> Net-(J30-Pin_2)
- U19 pad 11: Net-(J44-Pin_1) -> unconnected-(U19-Pad11)
- U19 pad 12: SLOPE_SW_RISE -> unconnected-(U19-Pad12)
- U19 pad 13: SLOPE_SW_FALL -> unconnected-(U19-Pad13)
- U19 pad 14: SLOPE_SW_OUT -> unconnected-(U19-Pad14)
- U19 pad 15: Net-(J43-Pin_6) -> Net-(J30-Pin_1)
- U19 pad 2: Net-(J43-Pin_2) -> Net-(J30-Pin_4)
- U19 pad 3: Net-(J43-Pin_3) -> Net-(J17-Pin_1)
- U19 pad 4: Net-(J43-Pin_4) -> ~{BOUNDS}
- U19 pad 5: Net-(J43-Pin_5) -> Net-(J16-Pin_1)
- U19 pad 9: A_SW -> DIRECTION
- U3 pad 10: LOGIC_S1 -> PENDULUM_MODE
- U3 pad 11: LOGIC_S2 -> ENV_MODE
- U3 pad 13: A_SW -> INV_DIRECTION
- U3 pad 14: Net-(U3-A) -> FILTER_CRITERIA
- U3 pad 15: Net-(U1B-C) -> MOVEMENT_TRIG
- U3 pad 2: ONESHOT_OR_RETRIG -> FILTERED_TRIG
- U3 pad 4: A_SW -> DIRECTION
- U3 pad 9: LOGIC_S3 -> GATE_MODE
- U4 pad 1: A0 -> -5V
- U4 pad 3: Net-(U4A-+) -> GND
- U4 pad 4: +12V -> -12V
- U4 pad 8: -12V -> +12V
- U7 pad 1: Net-(J18-Pin_2) -> Net-(JP6-A)
- U7 pad 2: B -> Net-(JP6-B)
- U7 pad 3: GND -> Net-(JP5-B)
- U7 pad 4: +12V -> -12V
- U7 pad 7: Net-(IC1A-CTRL) -> SLEW_CV
- U7 pad 8: -12V -> +12V
- U9 pad 11: +12V -> -12V
- U9 pad 4: -12V -> +12V
Routing:
- net A_SW: track 355.2 -> 0.00 mm, vias 8 -> 0
- net -5V: track 0.00 -> 293.2 mm, vias 0 -> 13
- net SYNC: track 276.2 -> 0.00 mm, vias 5 -> 0
- net A0: track 226.5 -> 0.00 mm, vias 10 -> 0
- net DIRECTION: track 0.00 -> 198.1 mm, vias 0 -> 4
- net AT_TARGET: track 168.7 -> 0.00 mm
- net ~{BOUNDS}: track 0.00 -> 122.5 mm
- net +12V: track 814.7 -> 695.5 mm, vias 17 -> 13
- net GND: track 233.4 -> 137.9 mm, vias 100 -> 54
- net 5VREF: track 188.0 -> 268.2 mm, vias 5 -> 8
- net EOC: track 268.9 -> 190.8 mm, vias 5 -> 1
- net SLOPE_FREQ_MOD: track 91.3 -> 15.4 mm, vias 1 -> 0
- net Net-(J18-Pin_2): track 76.5 -> 3.98 mm, vias 4 -> 0
- net B0: track 65.7 -> 0.00 mm
- net SLEW_CV: track 0.00 -> 63.1 mm, vias 0 -> 2
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Other:
- board text added: "ANALOG VIA V2"
- board text added: "G"
- board text added: "HOLD REF INV"
- board text added: "I"
- board text added: "O"
- board text removed: "ANALOG VIA V1"
- board text removed: "INPUT"
- board text removed: "S1 S2 S3"

Commit message: v2 routed, no drc yet
Parts:
- removed J67: Conn_01x01, Connector_PinHeader_2.54mm:PinHeader_1x01_P2.54mm_Vertical
- removed R11: 1K, Resistor_SMD:R_0805_2012Metric
- added ?: , , F.Cu at (217.5, 15.0)
- added ?: , , F.Cu at (19.4, 15.0)
- added ?: , , F.Cu at (217.5, 137.5)
- added ?: , , F.Cu at (19.4, 137.5)
- added REF**100: PinHeader_1x01_P2.54mm_Vertical, Connector_PinHeader_2.54mm:PinHeader_1x01_P2.54mm_Vertical, F.Cu at (90.7, 73.2)
- added REF**100: PinHeader_1x01_P2.54mm_Vertical, Connector_PinHeader_2.54mm:PinHeader_1x01_P2.54mm_Vertical, F.Cu at (182.5, 75.5)
- added REF**100: PinHeader_1x01_P2.54mm_Vertical, Connector_PinHeader_2.54mm:PinHeader_1x01_P2.54mm_Vertical, F.Cu at (100.9, 73.2)
- added REF**100: PinHeader_1x01_P2.54mm_Vertical, Connector_PinHeader_2.54mm:PinHeader_1x01_P2.54mm_Vertical, F.Cu at (111.1, 73.2)
- added REF**101: PinHeader_1x01_P2.54mm_Vertical, Connector_PinHeader_2.54mm:PinHeader_1x01_P2.54mm_Vertical, F.Cu at (128.8, 73.2)
- added REF**101: PinHeader_1x01_P2.54mm_Vertical, Connector_PinHeader_2.54mm:PinHeader_1x01_P2.54mm_Vertical, F.Cu at (185.1, 75.5)
- added REF**101: PinHeader_1x01_P2.54mm_Vertical, Connector_PinHeader_2.54mm:PinHeader_1x01_P2.54mm_Vertical, F.Cu at (93.3, 73.2)
- added REF**101: PinHeader_1x01_P2.54mm_Vertical, Connector_PinHeader_2.54mm:PinHeader_1x01_P2.54mm_Vertical, F.Cu at (103.4, 73.2)
- added REF**102: PinHeader_1x01_P2.54mm_Vertical, Connector_PinHeader_2.54mm:PinHeader_1x01_P2.54mm_Vertical, F.Cu at (113.6, 73.2)
- added REF**103: PinHeader_1x01_P2.54mm_Vertical, Connector_PinHeader_2.54mm:PinHeader_1x01_P2.54mm_Vertical, F.Cu at (116.1, 73.2)
- added REF**104: PinHeader_1x01_P2.54mm_Vertical, Connector_PinHeader_2.54mm:PinHeader_1x01_P2.54mm_Vertical, F.Cu at (118.7, 73.2)
- added REF**105: PinHeader_1x01_P2.54mm_Vertical, Connector_PinHeader_2.54mm:PinHeader_1x01_P2.54mm_Vertical, F.Cu at (169.8, 78.0)
- added REF**105: PinHeader_1x01_P2.54mm_Vertical, Connector_PinHeader_2.54mm:PinHeader_1x01_P2.54mm_Vertical, F.Cu at (78.0, 75.8)
- added REF**106: PinHeader_1x01_P2.54mm_Vertical, Connector_PinHeader_2.54mm:PinHeader_1x01_P2.54mm_Vertical, F.Cu at (172.4, 78.0)
- added REF**106: PinHeader_1x01_P2.54mm_Vertical, Connector_PinHeader_2.54mm:PinHeader_1x01_P2.54mm_Vertical, F.Cu at (80.6, 75.8)
- added REF**107: PinHeader_1x01_P2.54mm_Vertical, Connector_PinHeader_2.54mm:PinHeader_1x01_P2.54mm_Vertical, F.Cu at (83.1, 75.8)
- added REF**107: PinHeader_1x01_P2.54mm_Vertical, Connector_PinHeader_2.54mm:PinHeader_1x01_P2.54mm_Vertical, F.Cu at (174.9, 78.0)
- added REF**108: PinHeader_1x01_P2.54mm_Vertical, Connector_PinHeader_2.54mm:PinHeader_1x01_P2.54mm_Vertical, F.Cu at (202.8, 78.0)
- added REF**108: PinHeader_1x01_P2.54mm_Vertical, Connector_PinHeader_2.54mm:PinHeader_1x01_P2.54mm_Vertical, F.Cu at (177.4, 78.0)
- added REF**108: PinHeader_1x01_P2.54mm_Vertical, Connector_PinHeader_2.54mm:PinHeader_1x01_P2.54mm_Vertical, F.Cu at (85.7, 75.8)
- added REF**108: PinHeader_1x01_P2.54mm_Vertical, Connector_PinHeader_2.54mm:PinHeader_1x01_P2.54mm_Vertical, F.Cu at (95.8, 75.8)
- added REF**108: PinHeader_1x01_P2.54mm_Vertical, Connector_PinHeader_2.54mm:PinHeader_1x01_P2.54mm_Vertical, F.Cu at (106.0, 75.8)
- added REF**109: PinHeader_1x01_P2.54mm_Vertical, Connector_PinHeader_2.54mm:PinHeader_1x01_P2.54mm_Vertical, F.Cu at (180.0, 78.0)
- added REF**109: PinHeader_1x01_P2.54mm_Vertical, Connector_PinHeader_2.54mm:PinHeader_1x01_P2.54mm_Vertical, F.Cu at (98.4, 75.8)
- added REF**109: PinHeader_1x01_P2.54mm_Vertical, Connector_PinHeader_2.54mm:PinHeader_1x01_P2.54mm_Vertical, F.Cu at (88.2, 75.8)
- added REF**109: PinHeader_1x01_P2.54mm_Vertical, Connector_PinHeader_2.54mm:PinHeader_1x01_P2.54mm_Vertical, F.Cu at (108.5, 75.8)
- added REF**110: PinHeader_1x01_P2.54mm_Vertical, Connector_PinHeader_2.54mm:PinHeader_1x01_P2.54mm_Vertical, F.Cu at (100.9, 75.8)
- added REF**110: PinHeader_1x01_P2.54mm_Vertical, Connector_PinHeader_2.54mm:PinHeader_1x01_P2.54mm_Vertical, F.Cu at (111.1, 75.8)
- added REF**110: PinHeader_1x01_P2.54mm_Vertical, Connector_PinHeader_2.54mm:PinHeader_1x01_P2.54mm_Vertical, F.Cu at (90.7, 75.8)
- added REF**110: PinHeader_1x01_P2.54mm_Vertical, Connector_PinHeader_2.54mm:PinHeader_1x01_P2.54mm_Vertical, F.Cu at (182.5, 78.0)
- added REF**111: PinHeader_1x01_P2.54mm_Vertical, Connector_PinHeader_2.54mm:PinHeader_1x01_P2.54mm_Vertical, F.Cu at (103.4, 75.8)
- added REF**111: PinHeader_1x01_P2.54mm_Vertical, Connector_PinHeader_2.54mm:PinHeader_1x01_P2.54mm_Vertical, F.Cu at (185.1, 78.0)
- added REF**111: PinHeader_1x01_P2.54mm_Vertical, Connector_PinHeader_2.54mm:PinHeader_1x01_P2.54mm_Vertical, F.Cu at (93.3, 75.8)
- added REF**111: PinHeader_1x01_P2.54mm_Vertical, Connector_PinHeader_2.54mm:PinHeader_1x01_P2.54mm_Vertical, F.Cu at (128.8, 75.8)
- added REF**112: PinHeader_1x01_P2.54mm_Vertical, Connector_PinHeader_2.54mm:PinHeader_1x01_P2.54mm_Vertical, F.Cu at (113.6, 75.8)
- added REF**113: PinHeader_1x01_P2.54mm_Vertical, Connector_PinHeader_2.54mm:PinHeader_1x01_P2.54mm_Vertical, F.Cu at (116.1, 75.8)
- added REF**114: PinHeader_1x01_P2.54mm_Vertical, Connector_PinHeader_2.54mm:PinHeader_1x01_P2.54mm_Vertical, F.Cu at (118.7, 75.8)
- added REF**115: PinHeader_1x01_P2.54mm_Vertical, Connector_PinHeader_2.54mm:PinHeader_1x01_P2.54mm_Vertical, F.Cu at (169.8, 80.5)
- added REF**115: PinHeader_1x01_P2.54mm_Vertical, Connector_PinHeader_2.54mm:PinHeader_1x01_P2.54mm_Vertical, F.Cu at (78.0, 78.3)
- added REF**116: PinHeader_1x01_P2.54mm_Vertical, Connector_PinHeader_2.54mm:PinHeader_1x01_P2.54mm_Vertical, F.Cu at (172.4, 80.5)
- added REF**116: PinHeader_1x01_P2.54mm_Vertical, Connector_PinHeader_2.54mm:PinHeader_1x01_P2.54mm_Vertical, F.Cu at (80.6, 78.3)
- added REF**117: PinHeader_1x01_P2.54mm_Vertical, Connector_PinHeader_2.54mm:PinHeader_1x01_P2.54mm_Vertical, F.Cu at (83.1, 78.3)
- added REF**117: PinHeader_1x01_P2.54mm_Vertical, Connector_PinHeader_2.54mm:PinHeader_1x01_P2.54mm_Vertical, F.Cu at (174.9, 80.5)
- added REF**118: PinHeader_1x01_P2.54mm_Vertical, Connector_PinHeader_2.54mm:PinHeader_1x01_P2.54mm_Vertical, F.Cu at (85.7, 78.3)
- added REF**118: PinHeader_1x01_P2.54mm_Vertical, Connector_PinHeader_2.54mm:PinHeader_1x01_P2.54mm_Vertical, F.Cu at (95.8, 78.3)
- added REF**118: PinHeader_1x01_P2.54mm_Vertical, Connector_PinHeader_2.54mm:PinHeader_1x01_P2.54mm_Vertical, F.Cu at (177.4, 80.5)
- added REF**118: PinHeader_1x01_P2.54mm_Vertical, Connector_PinHeader_2.54mm:PinHeader_1x01_P2.54mm_Vertical, F.Cu at (202.8, 80.5)
- added REF**118: PinHeader_1x01_P2.54mm_Vertical, Connector_PinHeader_2.54mm:PinHeader_1x01_P2.54mm_Vertical, F.Cu at (106.0, 78.3)
- added REF**119: PinHeader_1x01_P2.54mm_Vertical, Connector_PinHeader_2.54mm:PinHeader_1x01_P2.54mm_Vertical, F.Cu at (180.0, 80.5)
- added REF**119: PinHeader_1x01_P2.54mm_Vertical, Connector_PinHeader_2.54mm:PinHeader_1x01_P2.54mm_Vertical, F.Cu at (108.5, 78.3)
- added REF**119: PinHeader_1x01_P2.54mm_Vertical, Connector_PinHeader_2.54mm:PinHeader_1x01_P2.54mm_Vertical, F.Cu at (98.4, 78.3)
- added REF**119: PinHeader_1x01_P2.54mm_Vertical, Connector_PinHeader_2.54mm:PinHeader_1x01_P2.54mm_Vertical, F.Cu at (88.2, 78.3)
- added REF**120: PinHeader_1x01_P2.54mm_Vertical, Connector_PinHeader_2.54mm:PinHeader_1x01_P2.54mm_Vertical, F.Cu at (182.5, 80.5)
- added REF**120: PinHeader_1x01_P2.54mm_Vertical, Connector_PinHeader_2.54mm:PinHeader_1x01_P2.54mm_Vertical, F.Cu at (111.1, 78.3)
- added REF**120: PinHeader_1x01_P2.54mm_Vertical, Connector_PinHeader_2.54mm:PinHeader_1x01_P2.54mm_Vertical, F.Cu at (90.7, 78.3)
- added REF**120: PinHeader_1x01_P2.54mm_Vertical, Connector_PinHeader_2.54mm:PinHeader_1x01_P2.54mm_Vertical, F.Cu at (100.9, 78.3)
- added REF**121: PinHeader_1x01_P2.54mm_Vertical, Connector_PinHeader_2.54mm:PinHeader_1x01_P2.54mm_Vertical, F.Cu at (103.4, 78.3)
- added REF**121: PinHeader_1x01_P2.54mm_Vertical, Connector_PinHeader_2.54mm:PinHeader_1x01_P2.54mm_Vertical, F.Cu at (185.1, 80.5)
- added REF**121: PinHeader_1x01_P2.54mm_Vertical, Connector_PinHeader_2.54mm:PinHeader_1x01_P2.54mm_Vertical, F.Cu at (93.3, 78.3)
- added REF**121: PinHeader_1x01_P2.54mm_Vertical, Connector_PinHeader_2.54mm:PinHeader_1x01_P2.54mm_Vertical, F.Cu at (128.8, 78.3)
- added REF**122: PinHeader_1x01_P2.54mm_Vertical, Connector_PinHeader_2.54mm:PinHeader_1x01_P2.54mm_Vertical, F.Cu at (113.6, 78.3)
- added REF**123: PinHeader_1x01_P2.54mm_Vertical, Connector_PinHeader_2.54mm:PinHeader_1x01_P2.54mm_Vertical, F.Cu at (116.1, 78.3)
- added REF**124: PinHeader_1x01_P2.54mm_Vertical, Connector_PinHeader_2.54mm:PinHeader_1x01_P2.54mm_Vertical, F.Cu at (118.7, 78.3)
- added REF**125: PinHeader_1x01_P2.54mm_Vertical, Connector_PinHeader_2.54mm:PinHeader_1x01_P2.54mm_Vertical, F.Cu at (169.8, 83.1)
- added REF**125: PinHeader_1x01_P2.54mm_Vertical, Connector_PinHeader_2.54mm:PinHeader_1x01_P2.54mm_Vertical, F.Cu at (95.8, 96.1)
- added REF**125: PinHeader_1x01_P2.54mm_Vertical, Connector_PinHeader_2.54mm:PinHeader_1x01_P2.54mm_Vertical, F.Cu at (78.0, 80.9)
- added REF**125: PinHeader_1x01_P2.54mm_Vertical, Connector_PinHeader_2.54mm:PinHeader_1x01_P2.54mm_Vertical, F.Cu at (202.8, 98.3)
- added REF**126: PinHeader_1x01_P2.54mm_Vertical, Connector_PinHeader_2.54mm:PinHeader_1x01_P2.54mm_Vertical, F.Cu at (172.4, 83.1)
- added REF**126: PinHeader_1x01_P2.54mm_Vertical, Connector_PinHeader_2.54mm:PinHeader_1x01_P2.54mm_Vertical, F.Cu at (80.6, 83.4)
- added REF**126: PinHeader_1x01_P2.54mm_Vertical, Connector_PinHeader_2.54mm:PinHeader_1x01_P2.54mm_Vertical, F.Cu at (172.4, 85.6)
- added REF**126: PinHeader_1x01_P2.54mm_Vertical, Connector_PinHeader_2.54mm:PinHeader_1x01_P2.54mm_Vertical, F.Cu at (80.6, 80.9)
- added REF**127: PinHeader_1x01_P2.54mm_Vertical, Connector_PinHeader_2.54mm:PinHeader_1x01_P2.54mm_Vertical, F.Cu at (83.1, 80.9)
- added REF**127: PinHeader_1x01_P2.54mm_Vertical, Connector_PinHeader_2.54mm:PinHeader_1x01_P2.54mm_Vertical, F.Cu at (83.1, 83.4)
- added REF**127: PinHeader_1x01_P2.54mm_Vertical, Connector_PinHeader_2.54mm:PinHeader_1x01_P2.54mm_Vertical, F.Cu at (174.9, 85.6)
- added REF**127: PinHeader_1x01_P2.54mm_Vertical, Connector_PinHeader_2.54mm:PinHeader_1x01_P2.54mm_Vertical, F.Cu at (174.9, 83.1)
- added REF**128: PinHeader_1x01_P2.54mm_Vertical, Connector_PinHeader_2.54mm:PinHeader_1x01_P2.54mm_Vertical, F.Cu at (85.7, 83.4)
- added REF**128: PinHeader_1x01_P2.54mm_Vertical, Connector_PinHeader_2.54mm:PinHeader_1x01_P2.54mm_Vertical, F.Cu at (202.8, 83.1)
- added REF**128: PinHeader_1x01_P2.54mm_Vertical, Connector_PinHeader_2.54mm:PinHeader_1x01_P2.54mm_Vertical, F.Cu at (177.4, 85.6)
- added REF**128: PinHeader_1x01_P2.54mm_Vertical, Connector_PinHeader_2.54mm:PinHeader_1x01_P2.54mm_Vertical, F.Cu at (95.8, 83.4)
- added REF**128: PinHeader_1x01_P2.54mm_Vertical, Connector_PinHeader_2.54mm:PinHeader_1x01_P2.54mm_Vertical, F.Cu at (95.8, 80.9)
- added REF**128: PinHeader_1x01_P2.54mm_Vertical, Connector_PinHeader_2.54mm:PinHeader_1x01_P2.54mm_Vertical, F.Cu at (177.4, 83.1)
- added REF**128: PinHeader_1x01_P2.54mm_Vertical, Connector_PinHeader_2.54mm:PinHeader_1x01_P2.54mm_Vertical, F.Cu at (85.7, 80.9)
- added REF**128: PinHeader_1x01_P2.54mm_Vertical, Connector_PinHeader_2.54mm:PinHeader_1x01_P2.54mm_Vertical, F.Cu at (202.8, 85.6)
- added REF**129: PinHeader_1x01_P2.54mm_Vertical, Connector_PinHeader_2.54mm:PinHeader_1x01_P2.54mm_Vertical, F.Cu at (88.2, 80.9)
- added REF**129: PinHeader_1x01_P2.54mm_Vertical, Connector_PinHeader_2.54mm:PinHeader_1x01_P2.54mm_Vertical, F.Cu at (180.0, 85.6)
- added REF**129: PinHeader_1x01_P2.54mm_Vertical, Connector_PinHeader_2.54mm:PinHeader_1x01_P2.54mm_Vertical, F.Cu at (98.4, 80.9)
- added REF**129: PinHeader_1x01_P2.54mm_Vertical, Connector_PinHeader_2.54mm:PinHeader_1x01_P2.54mm_Vertical, F.Cu at (180.0, 83.1)
- added REF**129: PinHeader_1x01_P2.54mm_Vertical, Connector_PinHeader_2.54mm:PinHeader_1x01_P2.54mm_Vertical, F.Cu at (98.4, 83.4)
- added REF**129: PinHeader_1x01_P2.54mm_Vertical, Connector_PinHeader_2.54mm:PinHeader_1x01_P2.54mm_Vertical, F.Cu at (88.2, 83.4)
- added REF**13: PinHeader_1x01_P2.54mm_Vertical, Connector_PinHeader_2.54mm:PinHeader_1x01_P2.54mm_Vertical, F.Cu at (78.0, 60.5)
- added REF**130: PinHeader_1x01_P2.54mm_Vertical, Connector_PinHeader_2.54mm:PinHeader_1x01_P2.54mm_Vertical, F.Cu at (90.7, 80.9)
- added REF**130: PinHeader_1x01_P2.54mm_Vertical, Connector_PinHeader_2.54mm:PinHeader_1x01_P2.54mm_Vertical, F.Cu at (182.5, 85.6)
- added REF**130: PinHeader_1x01_P2.54mm_Vertical, Connector_PinHeader_2.54mm:PinHeader_1x01_P2.54mm_Vertical, F.Cu at (90.7, 83.4)
- added REF**130: PinHeader_1x01_P2.54mm_Vertical, Connector_PinHeader_2.54mm:PinHeader_1x01_P2.54mm_Vertical, F.Cu at (100.9, 80.9)
- added REF**130: PinHeader_1x01_P2.54mm_Vertical, Connector_PinHeader_2.54mm:PinHeader_1x01_P2.54mm_Vertical, F.Cu at (100.9, 83.4)
- added REF**130: PinHeader_1x01_P2.54mm_Vertical, Connector_PinHeader_2.54mm:PinHeader_1x01_P2.54mm_Vertical, F.Cu at (182.5, 83.1)
- added REF**130: PinHeader_1x01_P2.54mm_Vertical, Connector_PinHeader_2.54mm:PinHeader_1x01_P2.54mm_Vertical, F.Cu at (111.1, 80.9)
- added REF**131: PinHeader_1x01_P2.54mm_Vertical, Connector_PinHeader_2.54mm:PinHeader_1x01_P2.54mm_Vertical, F.Cu at (128.8, 80.9)
- added REF**131: PinHeader_1x01_P2.54mm_Vertical, Connector_PinHeader_2.54mm:PinHeader_1x01_P2.54mm_Vertical, F.Cu at (185.1, 83.1)
- added REF**131: PinHeader_1x01_P2.54mm_Vertical, Connector_PinHeader_2.54mm:PinHeader_1x01_P2.54mm_Vertical, F.Cu at (103.4, 80.9)
- added REF**131: PinHeader_1x01_P2.54mm_Vertical, Connector_PinHeader_2.54mm:PinHeader_1x01_P2.54mm_Vertical, F.Cu at (93.3, 83.4)
- added REF**131: PinHeader_1x01_P2.54mm_Vertical, Connector_PinHeader_2.54mm:PinHeader_1x01_P2.54mm_Vertical, F.Cu at (185.1, 85.6)
- added REF**131: PinHeader_1x01_P2.54mm_Vertical, Connector_PinHeader_2.54mm:PinHeader_1x01_P2.54mm_Vertical, F.Cu at (93.3, 80.9)
- added REF**131: PinHeader_1x01_P2.54mm_Vertical, Connector_PinHeader_2.54mm:PinHeader_1x01_P2.54mm_Vertical, F.Cu at (103.4, 83.4)
- added REF**132: PinHeader_1x01_P2.54mm_Vertical, Connector_PinHeader_2.54mm:PinHeader_1x01_P2.54mm_Vertical, F.Cu at (169.8, 85.6)
- added REF**132: PinHeader_1x01_P2.54mm_Vertical, Connector_PinHeader_2.54mm:PinHeader_1x01_P2.54mm_Vertical, F.Cu at (78.0, 83.4)
- added REF**133: PinHeader_1x01_P2.54mm_Vertical, Connector_PinHeader_2.54mm:PinHeader_1x01_P2.54mm_Vertical, F.Cu at (95.8, 85.9)
- added REF**133: PinHeader_1x01_P2.54mm_Vertical, Connector_PinHeader_2.54mm:PinHeader_1x01_P2.54mm_Vertical, F.Cu at (202.8, 88.2)
- added REF**134: PinHeader_1x01_P2.54mm_Vertical, Connector_PinHeader_2.54mm:PinHeader_1x01_P2.54mm_Vertical, F.Cu at (202.8, 90.7)
- added REF**134: PinHeader_1x01_P2.54mm_Vertical, Connector_PinHeader_2.54mm:PinHeader_1x01_P2.54mm_Vertical, F.Cu at (95.8, 88.5)
- added REF**135: PinHeader_1x01_P2.54mm_Vertical, Connector_PinHeader_2.54mm:PinHeader_1x01_P2.54mm_Vertical, F.Cu at (202.8, 93.2)
- added REF**135: PinHeader_1x01_P2.54mm_Vertical, Connector_PinHeader_2.54mm:PinHeader_1x01_P2.54mm_Vertical, F.Cu at (95.8, 91.0)
- added REF**136: PinHeader_1x01_P2.54mm_Vertical, Connector_PinHeader_2.54mm:PinHeader_1x01_P2.54mm_Vertical, F.Cu at (95.8, 93.6)
- added REF**136: PinHeader_1x01_P2.54mm_Vertical, Connector_PinHeader_2.54mm:PinHeader_1x01_P2.54mm_Vertical, F.Cu at (202.8, 95.8)
- added REF**137: PinHeader_1x01_P2.54mm_Vertical, Connector_PinHeader_2.54mm:PinHeader_1x01_P2.54mm_Vertical, F.Cu at (169.8, 98.3)
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Connections:
- C33 pad 1: GND -> +12V
- C33 pad 2: -12V -> GND
- C7 pad 1: +12V -> GND
- C7 pad 2: GND -> -12V
- J60 pad 1: GND -> Net-(J60-Pin_1)
- J60 pad 2: unconnected-(J60-Pin_2-Pad2) -> Net-(J60-Pin_2)
- RV4 pad 1: +5V -> GND
- RV4 pad 3: GND -> +5V
- U39 pad 5: unconnected-(U39-Pad5) -> Net-(J29-Pin_2)
- U39 pad 6: unconnected-(U39-Pad6) -> Net-(J60-Pin_1)
- U39 pad 8: unconnected-(U39-Pad8) -> Net-(J60-Pin_2)
- U39 pad 9: unconnected-(U39-Pad9) -> Net-(J29-Pin_4)
- U9 pad 1: Net-(C8-Pad2) -> OUTPUT
- U9 pad 12: Net-(JP3-B) -> GND
- U9 pad 13: Net-(JP4-B) -> Net-(IC2C-OUT)
- U9 pad 14: Net-(JP4-A) -> Net-(C16-Pad2)
- U9 pad 2: Net-(IC2A-OUT) -> Net-(IC2B-OUT)
- U9 pad 5: GND -> Net-(JP3-B)
- U9 pad 6: Net-(IC2C-OUT) -> Net-(JP4-B)
- U9 pad 7: Net-(C16-Pad2) -> Net-(JP4-A)
- U9 pad 8: OUTPUT -> Net-(C8-Pad2)
- U9 pad 9: Net-(IC2B-OUT) -> Net-(IC2A-OUT)
Routing:
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- added copper zone on B.Cu, net +12V
- added copper zone on In2.Cu, net +12V
- added copper zone on In2.Cu, net +5V
- added copper zone on In2.Cu, net -12V
- added copper zone on In1.Cu, net GND
- removed copper zone on B.Cu, net GND
- removed copper zone on F.Cu, net GND
Other:
- copper layers 2 -> 4
- board text added: "CC BY-SA-NC 2025 Starling"
- board text added: "MODE SELECT"
- board text added: "S+H"
- board text added: "SERVO"
- board text added: "SYNC/ TRIG"
- board text added: "TRIG"
- board text removed: "2.5 VREF"
- board text removed: "CC BY-SA-NC 2024 Starling"
- board text removed: "CLK/2"
- board text removed: "CURRENT SOURCE"
- board text removed: "FLIP-FLOP TRIGGER"
- board text removed: "INTEGRATOR IN"
- board text removed: "INTEGRATOR OUT TO SLOPE"
- board text removed: "ONESHOT OR RETRIG"
- board text removed: "TRIGGER"

Commit message: v2 proto passes DRC
Parts:
- added J33: BOUNDS, Connector_PinHeader_2.00mm:PinHeader_1x01_P2.00mm_Vertical, F.Cu at (172.1, 124.8)
- added J34: GND, Connector_PinHeader_2.54mm:PinHeader_1x01_P2.54mm_Vertical, F.Cu at (114.2, 133.5)
- added J35: GND, Connector_PinHeader_2.54mm:PinHeader_1x01_P2.54mm_Vertical, F.Cu at (193.1, 117.9)
- added J43: GND, Connector_PinHeader_2.54mm:PinHeader_1x01_P2.54mm_Vertical, F.Cu at (38.7, 118.4)
- added J45: SPARE_OUT, Connector_PinHeader_2.54mm:PinHeader_1x01_P2.54mm_Vertical, F.Cu at (33.7, 87.5)
- added J46: GND, Connector_PinHeader_2.54mm:PinHeader_1x01_P2.54mm_Vertical, F.Cu at (148.4, 77.9)
- added J47: GND, Connector_PinHeader_2.54mm:PinHeader_1x01_P2.54mm_Vertical, F.Cu at (67.5, 30.5)
- added J48: +12V, Connector_PinHeader_2.54mm:PinHeader_1x01_P2.54mm_Vertical, F.Cu at (190.1, 101.0)
- added J49: -12V, Connector_PinHeader_2.54mm:PinHeader_1x01_P2.54mm_Vertical, F.Cu at (185.1, 101.0)
- added J51: +5V, Connector_PinHeader_2.54mm:PinHeader_1x01_P2.54mm_Vertical, F.Cu at (63.6, 85.0)
- added J52: +12V, Connector_PinHeader_2.54mm:PinHeader_1x01_P2.54mm_Vertical, F.Cu at (192.7, 101.0)
- added J53: -12V, Connector_PinHeader_2.54mm:PinHeader_1x01_P2.54mm_Vertical, F.Cu at (182.5, 101.0)
- added J54: +5V, Connector_PinHeader_2.54mm:PinHeader_1x01_P2.54mm_Vertical, F.Cu at (35.0, 118.4)
- added J55: GND, Connector_PinHeader_2.54mm:PinHeader_1x01_P2.54mm_Vertical, F.Cu at (180.0, 62.3)
- added J56: GND, Connector_PinHeader_2.54mm:PinHeader_1x01_P2.54mm_Vertical, F.Cu at (177.6, 62.3)
- added J57: GND, Connector_PinHeader_2.54mm:PinHeader_1x01_P2.54mm_Vertical, F.Cu at (174.9, 62.3)
- added J58: GND, Connector_PinHeader_2.54mm:PinHeader_1x01_P2.54mm_Vertical, F.Cu at (89.0, 53.4)
- added J59: GND, Connector_PinHeader_2.54mm:PinHeader_1x01_P2.54mm_Vertical, F.Cu at (91.7, 53.4)
- added J61: GND, Connector_PinHeader_2.54mm:PinHeader_1x01_P2.54mm_Vertical, F.Cu at (94.1, 53.4)
- added J62: INTEGRATOR_BUFFER, Connector_PinHeader_2.54mm:PinHeader_1x01_P2.54mm_Vertical, F.Cu at (133.8, 127.8)
- added J63: BIT1, Connector_PinHeader_2.54mm:PinHeader_1x01_P2.54mm_Vertical, F.Cu at (99.9, 122.4)
- added J66: BIT0, Connector_PinHeader_2.54mm:PinHeader_1x01_P2.54mm_Vertical, F.Cu at (96.0, 122.4)
- added J67: ENABLE_DECAY, Connector_PinHeader_2.54mm:PinHeader_1x01_P2.54mm_Vertical, F.Cu at (62.3, 91.7)
- added J68: AT_TARGET, Connector_PinHeader_2.00mm:PinHeader_1x01_P2.00mm_Vertical, F.Cu at (197.1, 118.0)
- added J69: EOA, Connector_PinHeader_2.54mm:PinHeader_1x01_P2.54mm_Vertical, F.Cu at (68.9, 86.5)
- added J70: DECAY_TRIG, Connector_PinHeader_2.54mm:PinHeader_1x01_P2.54mm_Vertical, F.Cu at (56.4, 109.6)
- added J71: DIR_CHANGE, Connector_PinHeader_2.54mm:PinHeader_1x01_P2.54mm_Vertical, F.Cu at (24.2, 112.1)
- added J72: MOVEMENT_TRIG, Connector_PinHeader_2.54mm:PinHeader_1x01_P2.54mm_Vertical, F.Cu at (47.3, 117.7)
- added J73: FILTERED_TRIG, Connector_PinHeader_2.54mm:PinHeader_1x01_P2.54mm_Vertical, F.Cu at (68.9, 91.6)
- added J74: FILTER_CRITERIA, Connector_PinHeader_2.54mm:PinHeader_1x01_P2.54mm_Vertical, F.Cu at (64.7, 118.4)
- J29: value Conn_02x02_Odd_Even -> GND; footprint Connector_PinHeader_2.54mm:PinHeader_2x02_P2.54mm_Vertical -> Connector_PinHeader_2.54mm:PinHeader_1x01_P2.54mm_Vertical
- J60: value Conn_01x02 -> SPARE_IN
- moved J29 11.3 mm to (44.9, 81.4), turned to 0 degrees
- moved J12 1.89 mm to (84.6, 122.0)
- moved J13 1.89 mm to (77.0, 119.5)
Connections:
- J60 pad 2: Net-(J60-Pin_2) -> GND
- U39 pad 5: Net-(J29-Pin_2) -> DIRECTION
- U39 pad 6: Net-(J60-Pin_1) -> INV_DIRECTION
- U39 pad 8: Net-(J60-Pin_2) -> Net-(J45-Pin_1)
- U39 pad 9: Net-(J29-Pin_4) -> Net-(J60-Pin_1)
Routing:
- net BIT1: track 14.0 -> 64.0 mm, vias 0 -> 1
- net BIT0: track 11.4 -> 55.7 mm, vias 0 -> 1
- net INV_DIRECTION: track 101.2 -> 143.5 mm
- net EOA: track 5.31 -> 30.4 mm, vias 0 -> 1
- net DIRECTION: track 324.0 -> 344.6 mm
- net 5VREF: track 252.8 -> 233.6 mm, vias 3 -> 1
- net FILTERED_TRIG: track 16.0 -> 31.7 mm, vias 0 -> 1
- net AT_TARGET: track 202.8 -> 217.5 mm
- net DIR_CHANGE: track 32.2 -> 43.6 mm
- net Net-(J29-Pin_2): track 11.0 -> 0.00 mm
- net Net-(J29-Pin_4): track 9.97 -> 0.00 mm, vias 1 -> 0
- net Net-(J60-Pin_2): track 8.81 -> 0.00 mm, vias 2 -> 0
- net FF_DIRECTION: track 54.3 -> 46.3 mm
- net ENABLE_DECAY: track 6.85 -> 14.3 mm, vias 0 -> 1
- net Net-(J60-Pin_1): track 8.98 -> 4.23 mm, vias 1 -> 0
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Other:
- board text added: "+5V"
- board text added: "0"
- board text added: "1"
- board text added: "2"
- board text added: "3"
- board text added: "A"
- board text added: "A/B"
- board text added: "AT TARGET"
- board text added: "B"
- board text added: "BIT0"
- board text added: "BIT1"
- board text added: "BOUNDARY"
- board text added: "BOUNDS"
- board text added: "BUF"
- board text added: "CTL"
- board text added: "DECAY TRIG"
- board text added: "DIR CHANGE"
- board text added: "ENABLE DECAY"
- board text added: "ENV"
- board text added: "EOA"
- board text added: "FC"
- board text added: "FF DIRECTION"
- board text added: "FILTERED TRIG"
- board text added: "FULL CYCLE"
- board text added: "GATE"
- board text added: "HOLD IN"
- board text added: "MODE"
- board text added: "MODE SEL"
- board text added: "MOVEMENT TRIG"
- board text added: "PENDULUM"
- board text removed: "1V/OCT"
- board text removed: "BOUNDARY COMPARATORS"
- board text removed: "MODE SELECT"
