File: analog-via.kicad_sch (KiCad schematic)
At the start: 209 parts, among them IC1 SSI2164, IC2 SSI2164, J1 2164_CV, J10 2164_IN, J11 SLEW_CV, J12 2164_CTL, J13 2164_OUT, J14 INTEGRATOR_IN, J15 COMP_CTL_A, J16 HIGH_COMP, J17 LOW_COMP, J18 INTEGRATOR, J19 OUTPUT, J2 5VREF, J20 COMP_CTL_B, J21 INV_SLOPE, J22 SLOPE, J23 POWER, J24 SYNC, J25 TRIGGER, J26 SYNC, J27 RISE, J28 FALL, J29 INA, J3 EXPO_IN, J30 INB, J31 OUTPUT, J32 DIRECTION, J33 EOC, J34 SLOPE, J35 CLK/2, J36 FALL_SUM, J37 RISE_SUM, J38 Conn_02x03_Counter_Clockwise, J39 2.5VREF, J4 FF_TRIGGER, J40 SLOPE_FREQ_MOD, J41 INA, J42 INB, J43 Conn_01x06, J44 EXTRA_SW_B, J45 EXTRA_SW_C, J46 LOGIC_S1, J47 LOGIC_S2, J48 LOGIC_S3, J49 Conn_01x03, J5 ONESHOT_OR_RETRIG, J50 1V/OCT, J6 TRIGGER, J7 EOC, J8 HOLD_REF, J9 INPUT, Q1 MMBFJ112, Q2 PNP, U1 74HC74, U10 DG333, U11 OPA1678, U12 LM311, U13 LM311, U14 OPA1678, U15 OPA1678, U16 TMUX4053PWR, U17 DG333, U18 AMS1117-5.0, U19 TMUX4053PWR, U2 LM4040DBZ-5, U3 TMUX4053PWR, U4 OPA1678, U5 LM339, U6 DG333, U7 OPA1678, U8 DG333, U9 OPA1679

Commit message: rotated op amp packages and corrected power supply issues, ratsnest still needs corrections
Parts:
- U2: JLCPCB C460604 -> C460606
Connections:
- net +12V: now also U11.8 (V+), U14.8 (V+), U15.8 (V+), U4.8 (V+), U7.8 (V+), U9.4 (V+); no longer U11.4 (V-), U14.4 (V-), U15.4 (V-), U4.4 (V-), U7.4 (V-), U9.11 (V-)
- net -12V: now also U11.4 (V-), U14.4 (V-), U15.4 (V-), U4.4 (V-), U7.4 (V-), U9.11 (V-); no longer U11.8 (V+), U14.8 (V+), U15.8 (V+), U4.8 (V+), U7.8 (V+), U9.4 (V+)
- net -5V: now also U4.7; no longer U4.1
- net B: now also U7.6 (-); no longer U7.2 (-)
- net GND: now also U11.3 (+), U11.5 (+), U14.3 (+), U14.5 (+), U15.5 (+), U7.3 (+), U7.5 (+), U9.10 (+), U9.12 (+), U9.5 (+); no longer U11.3 (+), U11.5 (+), U14.3 (+), U14.5 (+), U15.3 (+), U7.3 (+), U7.5 (+), U9.10 (+), U9.3 (+), U9.5 (+)
- net INV_SLOPE: now also U11.7; no longer U11.1
- net OUTPUT: now also U9.7; no longer U9.8
- net SLOPE: now also U11.1; no longer U11.7
- net SLOPE_FREQ_MOD: now also U15.7; no longer U15.1
- net SLOPE_SW_FALL: now also U14.1; no longer U14.7
- net SLOPE_SW_RISE: now also U14.7; no longer U14.1
- net at C3.2, IC1.3 (CTRL), IC1.6 (CTRL)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: now also U7.1; no longer U7.7
- net at R20.2: now also U4.5 (+); no longer U4.3 (+)
- net at R51.2, R52.1, R55.1: now also U11.6 (-); no longer U11.2 (-)
- net at C13.2, J18.2 (Pin_2), Q1.1 (D)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: now also U7.7; no longer U7.1
- net at C8.1, IC2.4 (OUT), R34.2: now also U9.13 (-); no longer U9.2 (-)
- net at C8.2, R38.2: now also U9.14; no longer U9.1
- net at R57.2, R59.1: now also U11.2 (-); no longer U11.6 (-)
- net at R69.2, R71.1: now also U15.6 (-); no longer U15.2 (-)
- net at C3.1, IC1.12 (OUT), J3.1 (Pin_1)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: now also U7.2 (-); no longer U7.6 (-)
- net at C16.1, IC2.12 (OUT), R46.2: now also U9.9 (-); no longer U9.6 (-)
- net at J36.1 (Pin_1), R61.2, R63.1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: now also U14.6 (-); no longer U14.2 (-)
- net at C16.2, R54.2: now also U9.8; no longer U9.7
- net at R21.1: now also U4.6 (-); no longer U4.2 (-)
- net at J37.1 (Pin_1), R62.2, R64.1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: now also U14.2 (-); no longer U14.6 (-)
- net at JP6.1 (A): now also U15.1; no longer U15.7
- net at JP6.2 (B): now also U15.2 (-); no longer U15.6 (-)
- net at JP2.1 (A): now also U4.1; no longer U4.7
- net at JP2.2 (B): now also U4.2 (-); no longer U4.6 (-)
- net at IC2.13 (OUT), IC2.5 (OUT), R47.1: now also U9.6 (-); no longer U9.9 (-)
- net at JP1.2 (B): now also U4.3 (+); no longer U4.5 (+)
- net at JP4.1 (A): now also U9.1; no longer U9.14
- net at JP4.2 (B): now also U9.2 (-); no longer U9.13 (-)
- net at JP5.2 (B): now also U15.3 (+); no longer U15.5 (+)
- net at JP3.2 (B): now also U9.3 (+); no longer U9.12 (+)
Other:
- note added: "EDIT: Changed part(typo) from 3V reference to 5V .2%"
