File: analog-via.kicad_sch (KiCad schematic)
At the start: 209 parts, among them IC1 SSI2164, IC2 SSI2164, J1 2164_CV, J10 2164_IN, J11 SLEW_CV, J12 2164_CTL, J13 2164_OUT, J14 INTEGRATOR_IN, J15 COMP_CTL_A, J16 HIGH_COMP, J17 LOW_COMP, J18 INTEGRATOR, J19 OUTPUT, J2 5VREF, J20 COMP_CTL_B, J21 INV_SLOPE, J22 SLOPE, J23 POWER, J24 SYNC, J25 TRIGGER, J26 SYNC, J27 RISE, J28 FALL, J29 INA, J3 EXPO_IN, J30 INB, J31 OUTPUT, J32 DIRECTION, J33 EOC, J34 SLOPE, J35 CLK/2, J36 FALL_SUM, J37 RISE_SUM, J38 Conn_02x03_Counter_Clockwise, J39 2.5VREF, J4 FF_TRIGGER, J40 SLOPE_FREQ_MOD, J41 INA, J42 INB, J43 Conn_01x06, J44 EXTRA_SW_B, J45 EXTRA_SW_C, J46 LOGIC_S1, J47 LOGIC_S2, J48 LOGIC_S3, J49 Conn_01x03, J5 ONESHOT_OR_RETRIG, J50 1V/OCT, J6 TRIGGER, J7 EOC, J8 HOLD_REF, J9 INPUT, Q1 MMBFJ112, Q2 PNP, U1 74HC74, U10 DG333, U11 OPA1678, U12 LM311, U13 LM311, U14 OPA1678, U15 OPA1678, U16 TMUX4053PWR, U17 DG333, U18 AMS1117-5.0, U19 TMUX4053PWR, U2 LM4040DBZ-5, U3 TMUX4053PWR, U4 OPA1678, U5 LM339, U6 DG333, U7 OPA1678, U8 DG333, U9 OPA1679

Commit message: pre-re-annotation, completed next rev schematic capture
Parts:
- removed C13: 1.2n, Capacitor_SMD:C_0805_2012Metric, symbol Device:C
- removed C23, C29: 100n, Capacitor_SMD:C_0805_2012Metric, symbol Device:C_Small
- removed C27, C28: 100p, Capacitor_SMD:C_0805_2012Metric, symbol Device:C
- removed D1, D2: 1N5819, Diode_SMD:D_SOD-123, symbol Device:D_Schottky
- removed J12: 2164_CTL, Connector_PinHeader_2.54mm:PinHeader_1x01_P2.54mm_Vertical, symbol Connector:Conn_01x01_Pin
- removed J13: 2164_OUT, Connector_PinHeader_2.54mm:PinHeader_1x01_P2.54mm_Vertical, symbol Connector:Conn_01x01_Pin
- removed J14: INTEGRATOR_IN, Connector_PinHeader_2.54mm:PinHeader_1x01_P2.54mm_Vertical, symbol Connector:Conn_01x01_Pin
- removed J18: INTEGRATOR, Connector_PinHeader_2.54mm:PinHeader_1x02_P2.54mm_Vertical, symbol Connector_Generic:Conn_01x02
- removed J24: SYNC, Connector_PinHeader_2.54mm:PinHeader_1x01_P2.54mm_Vertical, symbol Connector:Conn_01x01_Pin
- removed J38: Conn_02x03_Counter_Clockwise, symbol Connector_Generic:Conn_02x03_Counter_Clockwise
- removed J39: 2.5VREF, Connector_PinHeader_2.54mm:PinHeader_1x01_P2.54mm_Vertical, symbol Connector:Conn_01x01_Pin
- removed J49: Conn_01x03, Connector_PinHeader_2.54mm:PinHeader_1x03_P2.54mm_Vertical, symbol Connector_Generic:Conn_01x03
- removed J5: ONESHOT_OR_RETRIG, Connector_PinHeader_2.54mm:PinHeader_1x01_P2.54mm_Vertical, symbol Connector:Conn_01x01_Pin
- removed J6: TRIGGER, Connector_PinHeader_2.54mm:PinHeader_1x01_P2.54mm_Vertical, symbol Connector:Conn_01x01_Pin
- removed J7: EOC, Connector_PinHeader_2.54mm:PinHeader_1x01_P2.54mm_Vertical, symbol Connector:Conn_01x01_Pin
- removed J9: INPUT, Connector_Audio:Jack_3.5mm_QingPu_WQP-PJ398SM_Vertical_CircularHoles, symbol starling_symbols:Barrel_Jack_Switch
- removed Q1: MMBFJ112, Package_TO_SOT_SMD:SOT-23, symbol Transistor_FET:MMBFJ112
- removed Q2: PNP, Package_TO_SOT_SMD:SOT-23-3, symbol Simulation_SPICE:PNP
- removed R10, R5: 1M, Resistor_SMD:R_0805_2012Metric, symbol Device:R
- removed R11, R12, R13, R14, R15, R16, R66, R67, R68: 100k, Resistor_SMD:R_0805_2012Metric, symbol Device:R
- removed R17, R2, R22, R23, R45, R48, R65, R70, R8: 10k, Resistor_SMD:R_0805_2012Metric, symbol Device:R
- removed R27, R28, R29: 33k, Resistor_SMD:R_0805_2012Metric, symbol Device:R
- removed R60: 1k, Resistor_SMD:R_0805_2012Metric, symbol Device:R
- removed U10, U17, U6, U8: DG333, Package_SO:SOIC-20W_7.5x12.8mm_P1.27mm, symbol custom_ic:DG333
- removed U16, U19, U3: TMUX4053PWR, Package_SO:TSSOP-16_4.4x5mm_P0.65mm, symbol Analog_Switch:CD4053B
- removed U5: LM339, Package_SO:SOIC-14_3.9x8.7mm_P1.27mm, symbol Comparator:LM339
- removed unit 1 of U7
- added C47: 100p, Capacitor_SMD:C_0805_2012Metric, symbol Device:C
- added C48, C49: C_Small, symbol Device:C_Small
- added C50, C51: 1.2n, Capacitor_SMD:C_0805_2012Metric, symbol Device:C
- added C52: 1200p, Capacitor_SMD:C_0805_2012Metric, symbol Device:C_Small
- added C53: 1uF, symbol Device:C_Polarized
- added C54, C58, C59, C60, C61: 100n, Capacitor_SMD:C_0805_2012Metric, symbol Device:C_Small
- added C55: 100nF, symbol Device:C_Small
- added C56, C57: 100n, symbol Device:C_Small
- added D3: 1N5819, Diode_SMD:D_SOD-123, symbol Device:D_Schottky
- added D4: 1n4148, symbol Device:D
- added D5, D6, D7, D8: LED, symbol Device:LED
- added J12: Conn_02x04_Odd_Even, symbol Connector_Generic:Conn_02x04_Odd_Even
- added J13: Conn_01x04, symbol Connector_Generic:Conn_01x04
- added J18, J39: Conn_01x02_Pin, symbol Connector:Conn_01x02_Pin
- added J38: Conn_02x02_Counter_Clockwise, Connector_PinHeader_2.54mm:PinHeader_2x02_P2.54mm_Vertical, symbol Connector_Generic:Conn_02x02_Counter_Clockwise
- added J49, J53, J57, J59, J61, J63, J67: Conn_01x01, symbol Connector_Generic:Conn_01x01
- added J52: EXTRA_SW_B, Connector_PinHeader_2.54mm:PinHeader_1x01_P2.54mm_Vertical, symbol Connector:Conn_01x01_Pin
- added J54, J55, J56, J58, J60, J65: Conn_01x02, symbol Connector_Generic:Conn_01x02
- added J64: INV_HOLD_REF, Connector_PinHeader_2.54mm:PinHeader_1x01_P2.54mm_Vertical, symbol Connector:Conn_01x01_Pin
- added R100, R101, R98, R99: 1k, symbol Device:R
- added R102, R110, R94: 100k, symbol Device:R
- added R103, R83: 10k, Resistor_SMD:R_0805_2012Metric, symbol Device:R
- added R104, R107, R84: 100k, Resistor_SMD:R_0805_2012Metric, symbol Device:R
- added R105, R86: 1M, Resistor_SMD:R_0805_2012Metric, symbol Device:R
- added R106, R87: 4.7k, Resistor_SMD:R_0805_2012Metric, symbol Device:R
- added R108, R88, R89: 1M, symbol Device:R
- added R109: 1, symbol Device:R
- added R82, R85: 200k, symbol Device:R
- added R90: 33k, Resistor_SMD:R_0805_2012Metric, symbol Device:R
- added R91: 220, Resistor_SMD:R_0805_2012Metric, symbol Device:R
- added R92: 845, Resistor_SMD:R_0805_2012Metric, symbol Device:R
- added R93: 150k, symbol Device:R
- added R95, R96: 300k, symbol Device:R
- added R97: 600k, symbol Device:R
- added RV4: 100k, symbol Device:R_Potentiometer
- added U10: 74LS08, symbol 74xx:74LS08
- added U16, U19, U3, U6: TMUX4053, Package_SO:SOIC-20W_7.5x12.8mm_P1.27mm, symbol custom_ic:TMUX4053
- added U17: LM319, symbol Comparator:LM319
- added U22: 74AHC1G32, Package_TO_SOT_SMD:SOT-23-5, symbol 74xGxx:74AHC1G32
- added U30: 74AHC1G86, Package_TO_SOT_SMD:SOT-353_SC-70-5, symbol 74xGxx:74AHC1G86
- added U31, U38, U8: LM3900, symbol custom_ic:LM3900
- added U32: LF398_SOIC14, Package_SO:SOIC-14_3.9x8.7mm_P1.27mm, symbol custom_ic:LF398_SOIC14
- added U33, U34, U35, U36: OPA1678, symbol Amplifier_Operational:OPA1678
- added U37: TL431DBZ, Package_TO_SOT_SMD:SOT-23, symbol Reference_Voltage:TL431DBZ
- added U39, U40: 74HC14, symbol 74xx:74HC14
- added U42: 74HC237, symbol 74xx:74HC237
- J10: value 2164_IN -> TRIGGER
- J16: value HIGH_COMP -> LOW_COMP
- J17: value LOW_COMP -> HIGH_COMP
- J44: value EXTRA_SW_B -> ~{SYNC}
- R18: value 100k 1% -> 100k; footprint Resistor_SMD:R_0805_2012Metric -> (none)
- R19: value 100k 1% -> 150k; footprint Resistor_SMD:R_0805_2012Metric -> (none)
- R40, R41: value 1M -> DNP
- R69: value 100k -> 10M; footprint Resistor_SMD:R_0805_2012Metric -> (none); JLC (none) -> C7250
- R71: value 100k -> 33k
Connections:
- net A is gone; now on net HOLD_REF: J8.1 (Pin_1)
- net SLOPE_SW_OUT is gone; now on an unnamed net: R69.1
- net SYNC is gone; now on net +5V: U1.13 (~{R})
- net +12V: now also J23.10 (Pin_10), J23.9 (Pin_9), R1.2, U11.8 (V+), U14.8 (V+), U15.8 (V+), U4.8 (V+), U7.8 (V+), U9.4 (V+), C49.1, C54.1, C58.1, R92.1, U16.16 (VDD), U17.11 (V+), U19.16 (VDD), U3.16 (VDD), U32.12 (V+); no longer J23.1 (Pin_1), J23.2 (Pin_2), R1.1, U11.4 (V-), U14.4 (V-), U15.4 (V-), U4.4 (V-), U7.4 (V-), U9.11 (V-)
- net +5V: now also R36.1, C55.1, C56.1, C57.1, C60.1, C61.1, J13.1 (Pin_1), J13.2 (Pin_2), J13.3 (Pin_3), J13.4 (Pin_4), R104.2, R106.1, R109.2, R84.2, R87.1, R96.2, R97.2, RV4.1, U22.5 (VCC), U30.5 (VCC), U39.14 (VCC), U40.14 (VCC), U42.16 (VCC), U42.6 (E2), U8.14 (VCC); no longer U18.2 (VO)
- net -12V: now also C31.2, C44.2, J23.1 (Pin_1), J23.2 (Pin_2), U11.4 (V-), U14.4 (V-), U15.4 (V-), U4.4 (V-), U7.4 (V-), U9.11 (V-), C48.1, C59.2, U16.7 (VEE), U17.6 (V-), U19.7 (VEE), U32.3 (V-); no longer C31.1, C44.1, J23.10 (Pin_10), J23.9 (Pin_9), U11.8 (V+), U14.8 (V+), U15.8 (V+), U4.8 (V+), U7.8 (V+), U9.4 (V+)
- net -5V: now also RV2.1, RV3.1, U16.12, U16.2
- net 5VREF: now also U13.3 (-), C53.1, R92.2, U16.1, U16.13; no longer C1.1, R1.2, R18.2, R36.1, R44.2, R6.1
- net AT_TARGET: now also U1.5 (Q), U12.6 (STRB), U13.6 (STRB), J65.2 (Pin_2), U10.10, U10.2, U6.11; no longer R36.2
- net CLK/2: no longer U1.5 (Q)
- net EOC: now also U10.8, U3.12
- net GND: now also C31.1, C44.1, R69.2, U1.2 (D), U1.3 (C), U4.3 (+), C48.2, C49.2, C50.1, C52.1, C53.2, C54.2, C55.2, C56.2, C57.2, C58.2, C59.1, C60.2, C61.2, D5.1 (K), D6.1 (K), D7.1 (K), D8.1 (K), J54.1 (Pin_1), J55.1 (Pin_1), J56.1 (Pin_1), J58.1 (Pin_1), J60.1 (Pin_1), R102.1, R103.1, R108.2, R110.1, R83.1, R88.2, RV4.3, U16.6 (~{EN}), U16.8 (VSS), U17.3 (GND), U17.8 (GND), U19.6 (~{EN}), U19.8 (VSS), U22.3 (GND), U3.6 (~{EN}), U3.7 (VEE), U3.8 (VSS), U30.3 (GND), U32.10 (T), U34.3 (+), U35.3 (+), U37.3 (A), U39.7 (GND), U40.7 (GND), U42.3 (A2), U42.4 (~{LE}), U42.5 (~{E1}), U42.8 (GND), U8.7 (GND); no longer C31.2, C44.2, R19.1, RV2.1, RV3.1
- net SLOPE_FREQ_MOD: now also U19.14; no longer R71.2, U15.1
- net SYNC_IN: now also U17.5 (-)
- net TRIGGER: now also J10.1 (Pin_1), R105.2, R106.2, U10.12, U17.7, U3.1, U3.3
- net TRIGGER_IN: now also R107.1, R108.1
- net SLEW_CV: now reaches C3.2, IC1.3 (CTRL), IC1.6 (CTRL), J11.1 (Pin_1), RV1.2, RV1.3, U7.7
- net SLEW_CV: now also IC1.14 (CTRL)
- net at R20.2: now also R21.1, U4.2 (-); no longer U4.3 (+)
- net at U12.3 (-): now also R44.1, R51.1, J38.1 (Pin_1), J38.2 (Pin_2); no longer U13.3 (-)
- net ~{SYNC}: now reaches U1.10 (~{S})
- net ~{SYNC}: now also J44.1 (Pin_1), U40.2
- net DIR_CHANGE: now reaches U1.11 (C)
- net DIR_CHANGE: now also U22.4, U6.5
- net at R41.2, U13.2 (+): now also R44.2; no longer R44.1
- net HOLD_REF: now reaches R30.1
- net HOLD_REF: now also U16.14, U32.1 (I), U36.3 (+)
- net at IC1.13 (OUT): now also U6.12
- net at IC1.15 (IN): now also R71.2, R91.2; no longer J10.1 (Pin_1)
- net at J45.1 (Pin_1): now also U19.9
- net at J43.1 (Pin_1): now also U19.1
- net at J43.6 (Pin_6): now also U19.4
- net at J43.2 (Pin_2): now also U19.2
- net at J43.3 (Pin_3): now also U19.5
- net at J43.4 (Pin_4): now also U19.15
- net at J43.5 (Pin_5): now also U19.3
- net ACTIVATION_TRIG: now reaches U1.1 (~{R})
- net ACTIVATION_TRIG: now also U6.4
- net at U1.6 (~{Q}): no longer U1.2 (D)
- net ~{BOUNDS}: now reaches U1.4 (~{S})
- net ~{BOUNDS}: now also R36.2, U16.4
- net 2.5VREF: no longer names the net of R19.2
- net 2.5VREF: now also R18.2, U8.1 (+); no longer R18.1
- net A_SW renamed DIRECTION
- net DIRECTION: now also U10.1, U16.11, U16.9, U19.11, U3.4, U39.13; no longer U1.3 (C)
- net B0: no longer names the net of IC1.4 (OUT)
- net B0: now also R90.2, U34.2 (-)
- net C0: no longer names the net of J16.1 (Pin_1), R40.1, U12.7
- net C0: now also U16.5
- net C1: no longer names the net of J17.1 (Pin_1), R41.1, U13.7
- net C1: now also U16.3
- net FF_TRIGGER renamed FF_DIRECTION
- net FF_DIRECTION: now also U3.5
- net LOGIC_S1 renamed ENV_MODE
- net ENV_MODE: now also J12.3 (Pin_3), U3.11
- net LOGIC_S2 renamed PENDULUM_MODE
- net PENDULUM_MODE: now also J12.5 (Pin_5), U3.10
- net LOGIC_S3 renamed GATE_MODE
- net GATE_MODE: now also J12.7 (Pin_7), U3.9, U6.9
- net SLOPE_SW_FALL: no longer names the net of R64.2, U14.7
- net SLOPE_SW_FALL: now also U19.13
- net SLOPE_SW_RISE: no longer names the net of R63.2, U14.1
- net SLOPE_SW_RISE: now also U19.12
- new net: J67.1 (Pin_1), U39.10
- new net: R103.2, R104.1, U17.10 (-)
- new net: R105.1, R107.2, U17.9 (+)
- new net: D6.2 (A), R99.1
- new net: D4.1 (K), R97.1, U8.3 (-)
- new net: R86.2, R87.2, U17.12, U40.3
- new net: D5.2 (A), R98.1
- new net: R83.2, R84.1, R86.1, U17.4 (+)
- new net: C47.1, D3.2 (A), R102.2
- new net: C47.2, U40.4
- new net: J56.2 (Pin_2), U40.11
- new net: C51.1, U35.2 (-), U6.14
- new net: D4.2 (A), R95.1
- new net: J59.1 (Pin_1), U40.8
- new net: J61.1 (Pin_1), U40.10
- new net: J60.2 (Pin_2), U39.11
- new net: R89.2, R90.1, U34.1
- new net: D3.1 (K), R110.2, U40.1
- new net: J49.1 (Pin_1), J53.1 (Pin_1), U15.1, U15.2 (-)
- new net: R82.2, R85.2, U33.1
- new net: R85.1, R89.1, U33.2 (-)
- new net: C50.2, R82.1, R88.1, U32.8 (Ch), U33.3 (+)
- new net: J54.2 (Pin_2), U40.5
- new net: J57.1 (Pin_1), U40.6
- new net: J52.1 (Pin_1), U19.10
- new net: D7.2 (A), R100.1
- new net: J58.2 (Pin_2), U40.13
- new net: R93.2, R94.2, U8.2 (+)
- new net: C52.2, R91.1
- new net: J39.2 (Pin_2), U30.2
- new net: J39.1 (Pin_1), U39.8
- new net: J63.1 (Pin_1), U40.12
- new net: J18.2 (Pin_2), U39.1
- new net: U39.2, U39.3
- new net: C1.1, R1.1, R6.1, U37.1 (K), U37.2 (REF)
- new net: U36.1, U6.13
- new net: R19.1, R93.1, RV4.2
- new net: J65.1 (Pin_1), U32.11 (Hold)
- new net: U39.6, U39.9
- new net: R96.1, U8.6 (-)
- new net: U39.4, U39.5
- new net: D8.2 (A), R101.1
- new net: J55.2 (Pin_2), U40.9
- new net: R109.1, U18.2 (VO)
- new net BIT0: U42.1 (A0), U8.4
- new net BIT1: R95.2, U42.2 (A1), U8.5
- new net DECAY_TRIG: U10.6, U22.2
- new net ENABLE_DECAY: U10.4
- new net EOA: U10.3, U10.5
- new net FILTERED_TRIG: U10.11, U3.2
- new net FILTER_CRITERIA: U10.13, U3.14
- new net FULL_CYCLE_MODE: J12.1 (Pin_1)
- new net GATE: J18.1 (Pin_1), U30.1
- new net GATE_EDGE_TRIG: U30.4, U6.3
- new net HOLD_REF_INV: R71.1
- new net INTEGRATOR_II_OUT: C51.2, J38.3 (Pin_3), U35.1, U36.2 (-)
- new net INV_DIRECTION: U10.9, U16.10, U3.13, U39.12
- new net INV_HOLD_REF: J64.1 (Pin_1), U16.15
- new net MODE0: J12.2 (Pin_2), R98.2, U42.12 (Y3)
- new net MODE1: J12.4 (Pin_4), R99.2, U42.13 (Y2)
- new net MODE2: J12.6 (Pin_6), R100.2, U42.14 (Y1)
- new net MODE3: J12.8 (Pin_8), R101.2, U42.15 (Y0)
- new net MODE_CV: R18.1, R94.1
- new net MOVEMENT_TRIG: U22.1, U3.15
- new net S+H_INTEGRATOR_OUT: J38.4 (Pin_4), U32.7
- no-connect marks 5 -> 13
Other:
- note added: "20nS MINIMUM"
- note added: "ALL MODES OFF IS "FULL CYLCLE MODE""
- note added: "BOUNDS DETECTION AND SLOPE BUFFERING"
- note added: "CALCULATE HYSTERESIS/INPUT RESISTANCE"
- note added: "CALCULATE RESISTANCES FOR FEEDBACK NETWORK"
- note added: "CROSSFADER"
- note added: "Can this be +5V?"
- note added: "ENABLE DECAY is a mode switch DECAY_TRIG will cause a slope down immediately from 5V"
- note added: "EXPO CONVERTER/SLEW CV GENERATOR"
- note added: "EXTRA INVERTERS"
- note added: "FILTER_CRITERIA is a mode-dependent mechanism for choosing relevant triggers Either EOC or INV_DIRECTION"
- note added: "HOLD-> AT_TARGET OR !SYNC?"
- note added: "I/O"
- note added: "MODE SELECT"
- note added: "MOVEMENT_TRIG is the product of the switch network e.g. in pendulum mode, every external trig is a MOVEMENT_TRIG for the two "trigger modes", MOVEMENT_TRIG is the external trig filtered by the slope generator's state."
- note added: "NEED ENABLE_DECAY"
- note added: "POWER"
- note added: "REFERENCE VOLTAGES"
- note added: "RISE/FALL CV INPUT AND SWITCHING"
- note added: "S+H INTEGRATOR"
- note added: "SERVO INTEGRATOR"
- note added: "SYNC"
- note added: "SYNC pulse should also assert AT_TARGET?"
- note added: "TODO!!!"
- note added: "TODO: input resistors scaling"
- note added: "TRIGGER"
- note added: "bounds active low"
- note added: "exponential converter temperature compensated"
- note added: "https://tinyurl.com/24ptj5km"
- note added: "https://tinyurl.com/26u8mvxu"
- note added: "tantalum"
- note removed: "1.2n = 10kHz @ 5V -> 33k -> .15mA"
- note removed: "10uS input time constant"
- note removed: "1uS reset - could be as low as 300nS if desired?"
- note removed: "DUPLICATED ON OTHER SECTION"
- note removed: "HOLDING REFERENCE VOLTAGE"
- note removed: "INTEGRATOR"
- note removed: "SHOULD BE +5V NET THIS IS A HACK"
- note removed: "SHOULD GET LM339B for testing -- lower propagation delay"
- note removed: "SLEWING CURRENT"
- note removed: "SYNC PULSE SHAPER"
- note removed: "THIS WILL SHORT ON PLUG INSERT"
- note removed: "WHAT HAPPENS TO FLIP FLOP ON STARTUP"
- note removed: "When S3 is high, others are off, gate mode is on. When S2 is high, others are off, pendulum mode happens, every trigger switches direction When S1 is high, others are assumed off, triggers are ignored during attack When all switches are off, triggers are ignored until we reach the end of cycle"
- note removed: "exponential converter / temperature compensated"
- note removed: "https://tinyurl.com/27lmfat4"
- note removed: "or 5V?"
- moved on the sheet: C1, C10, C11, C12, C14, C15, C16, C17, C18, C19, C2, C20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

Commit message: routing
Parts:
- removed C14, C36: 100n, Capacitor_SMD:C_0805_2012Metric, symbol Device:C_Small
- removed J43: Conn_01x06, Connector_PinHeader_2.54mm:PinHeader_1x06_P2.54mm_Vertical, symbol Connector_Generic:Conn_01x06
- removed J45: EXTRA_SW_C, Connector_PinHeader_2.54mm:PinHeader_1x01_P2.54mm_Vertical, symbol Connector:Conn_01x01_Pin
- removed J46: LOGIC_S1, Connector_PinHeader_2.54mm:PinHeader_1x01_P2.54mm_Vertical, symbol Connector:Conn_01x01_Pin
- removed J47: LOGIC_S2, Connector_PinHeader_2.54mm:PinHeader_1x01_P2.54mm_Vertical, symbol Connector:Conn_01x01_Pin
- removed J48: LOGIC_S3, Connector_PinHeader_2.54mm:PinHeader_1x01_P2.54mm_Vertical, symbol Connector:Conn_01x01_Pin
- removed J49, J53, J57, J59, J61, J63: Conn_01x01, symbol Connector_Generic:Conn_01x01
- removed J52: EXTRA_SW_B, Connector_PinHeader_2.54mm:PinHeader_1x01_P2.54mm_Vertical, symbol Connector:Conn_01x01_Pin
- removed J54, J55, J56, J58: Conn_01x02, symbol Connector_Generic:Conn_01x02
- removed U15: OPA1678, Package_SO:SOIC-8_3.9x4.9mm_P1.27mm, symbol Amplifier_Operational:TL072
- added C13, C23, C27, C28, C46, C62: 100n, Capacitor_SMD:C_0805_2012Metric, symbol Device:C_Small
- added J30, J31: Conn_01x04, Connector_PinHeader_2.54mm:PinHeader_1x04_P2.54mm_Vertical, symbol Connector_Generic:Conn_01x04
- added J32: Conn_02x04_Odd_Even, Connector_PinHeader_2.54mm:PinHeader_2x04_P2.54mm_Vertical, symbol Connector_Generic:Conn_02x04_Odd_Even
- added unit 5 of U10
- added unit 3 of U33
- added unit 3 of U35
- added unit 1 of U7
- C48, C49: value C_Small -> 100n
- C53, C55: footprint (none) -> Capacitor_SMD:C_0805_2012Metric
- D4: footprint (none) -> Diode_SMD:D_SOD-123
- D5, D6, D7, D8: footprint (none) -> LED_SMD:LED_0805_2012Metric
- J12: footprint (none) -> Connector_PinHeader_2.54mm:PinHeader_2x04_P2.54mm_Vertical
- J13: footprint (none) -> Connector_PinHeader_2.54mm:PinHeader_1x04_P2.54mm_Vertical
- J18, J39, J60, J65: footprint (none) -> Connector_PinHeader_2.54mm:PinHeader_1x02_P2.54mm_Vertical
- J4: value FF_TRIGGER -> FF_DIRECTION
- J64: value INV_HOLD_REF -> HOLD_REF_INV
- J67: footprint (none) -> Connector_PinHeader_2.54mm:PinHeader_1x01_P2.54mm_Vertical
- R100, R101, R102, R108, R109, R110, R18, R19, R69, R82, R85, R93, R94, R95, R96, R97, R98, R99: footprint (none) -> Resistor_SMD:R_0805_2012Metric
- RV4: footprint (none) -> Potentiometer_THT:Potentiometer_TT_P0915N
- U10, U17, U39, U40, U8: footprint (none) -> Package_SO:SOIC-14_3.9x8.7mm_P1.27mm
- U16, U19, U3, U6: footprint Package_SO:SOIC-20W_7.5x12.8mm_P1.27mm -> Package_SO:TSSOP-16_4.4x5mm_P0.65mm
- U33, U35: footprint (none) -> Package_SO:SOIC-8_3.9x4.9mm_P1.27mm
- U33: renamed from U34; footprint (none) -> Package_SO:SOIC-8_3.9x4.9mm_P1.27mm
- U35: renamed from U36; footprint (none) -> Package_SO:SOIC-8_3.9x4.9mm_P1.27mm
- U42: footprint (none) -> Package_SO:SOIC-16_4.55x10.3mm_P1.27mm
- U8: renamed from U31; footprint (none) -> Package_SO:SOIC-14_3.9x8.7mm_P1.27mm
- U8: renamed from U38; footprint (none) -> Package_SO:SOIC-14_3.9x8.7mm_P1.27mm
- renumbered J30 to J14, J25 to J24, J26 to J25, J27 to J26, J28 to J27, J29 to J28, J35 to J29, J34 to J5, J33 to J6, J31 to J7, J32 to J9, R75 to R10, R73 to R11, R72 to R2, R74 to R5, R50 to R8
Connections:
- net INV_HOLD_REF is gone; now on net HOLD_REF_INV: J64.1 (Pin_1), U16.15
- net +12V: now also C23.1, C28.1, U33.8 (V+), U35.8 (V+)
- net +5V: now also C13.1, C27.1, U10.14 (VCC); no longer RV2.3, RV3.3
- net -12V: now also C46.2, C62.2, U33.4 (V-), U35.4 (V-)
- net 5VREF: now also RV2.3, RV3.3
- net DIRECTION: now also U19.9; no longer U19.11, U39.13
- net GND: now also U33.5 (+), C13.2, C23.2, C27.2, C28.2, C46.1, C62.1, J32.1 (Pin_1), J32.3 (Pin_3), J32.5 (Pin_5), J32.7 (Pin_7), U10.7 (GND); no longer U33.3 (+)
- net HOLD_REF: now also U35.5 (+); no longer U35.3 (+)
- net INTEGRATOR_II_OUT: now also U35.6 (-); no longer U35.2 (-)
- net INV_DIRECTION: no longer U39.12
- net SLOPE_FREQ_MOD: now also U16.4; no longer U19.14
- net ~{BOUNDS}: now also U19.4; no longer U16.4
- net at J67.1 (Pin_1): no longer U39.10
- net at J16.1 (Pin_1), R40.1, U12.7: now also U19.5; no longer U16.5
- net at IC1.4 (OUT), R90.2: now also U33.6 (-); no longer U33.2 (-)
- net at U40.11: now also J32.6 (Pin_6)
- net at U40.8: now also J31.2 (Pin_2)
- net at U40.10: now also J31.3 (Pin_3)
- net at U39.11: now also U39.4; no longer J60.2 (Pin_2)
- net at R89.2, R90.1: now also U33.7; no longer U33.1
- net at J17.1 (Pin_1), R41.1, U13.7: now also U19.3; no longer U16.3
- net at R64.2, U14.7: now also U16.3; no longer U19.13
- net at U40.5: now also J32.2 (Pin_2)
- net at U40.6: now also J31.1 (Pin_1)
- net at JP6.1 (A): now also U7.1
- net at JP6.2 (B): now also U7.2 (-)
- net at U19.1: now also J30.3 (Pin_3)
- net at U19.10: now also J30.2 (Pin_2)
- net at U19.15: now also J30.1 (Pin_1)
- net at U19.2: now also J30.4 (Pin_4)
- net at U40.13: now also J32.8 (Pin_8)
- net at R63.2, U14.1: now also U16.5; no longer U19.12
- net at J39.1 (Pin_1): now also U39.12; no longer U39.8
- net at U40.12: now also J31.4 (Pin_4)
- net at U6.13: now also U35.7; no longer U35.1
- net at U39.9: no longer U39.6
- net at U39.5: no longer U39.4
- net at U40.9: now also J32.4 (Pin_4)
- net at JP5.2 (B): now also U7.3 (+)
- new net: U39.10, U39.13
Other:
- note added: "AND mode logic"
- note added: "FULL_CYCLE_MODE does nothing"
- note added: "Move switch before opamps?"
- note added: "crossfader"
- note added: "delay lines/dir inv/sync"
- note added: "expo"
- note added: "flip flop mode logic"
- note added: "logic"
- note added: "mode sel"
- note added: "reference"
- note added: "reference/bounds"
- note added: "rise/fall"
- note added: "rise/fall cv"
- note added: "s+h integrator"
- note added: "servo integrator"
- note added: "slope"
- note added: "trig/sync"
- note removed: "NEED SWITCH HERE!!"
- note removed: "TODO!!!"
- moved on the sheet: C11, C15, C24, C32, C33, C34, C35, C37, C4, C48, C49, C5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
