File: analog-via.kicad_sch (KiCad schematic)
At the start: 231 parts, among them IC1 SSI2164, IC2 SSI2164, J1 2164_CV, J10 TRIGGER, J11 SLEW_CV, J12 Conn_02x04_Odd_Even, J13 Conn_01x04, J14 INB, J15 COMP_CTL_A, J16 LOW_COMP, J17 HIGH_COMP, J18 Conn_01x02_Pin, J19 OUTPUT, J2 5VREF, J20 COMP_CTL_B, J21 INV_SLOPE, J22 SLOPE, J23 POWER, J24 TRIGGER, J25 SYNC, J26 RISE, J27 FALL, J28 INA, J29 Conn_02x02_Odd_Even, J3 EXPO_IN, J30 Conn_01x04, J31 Conn_01x04, J32 Conn_02x04_Odd_Even, J36 FALL_SUM, J37 RISE_SUM, J38 Conn_02x02_Counter_Clockwise, J39 Conn_01x02_Pin, J4 FF_DIRECTION, J40 SLOPE_FREQ_MOD, J41 INA, J42 INB, J44 ~{SYNC}, J5 SLOPE, J50 1V/OCT, J6 EOC, J60 Conn_01x02, J64 HOLD_REF_INV, J65 Conn_01x02, J7 OUTPUT, J8 HOLD_REF, J9 DIRECTION, U1 74HC74, U10 74LS08, U11 OPA1678, U12 LM311, U13 LM311, U14 OPA1678, U16 TMUX4053, U17 LM319, U18 AMS1117-5.0, U19 TMUX4053, U2 LM4040DBZ-5, U22 74AHC1G32, U3 TMUX4053, U30 74AHC1G86, U32 LF398_SOIC14, U33 OPA1678, U35 OPA1678, U37 TL431DBZ, U39 74HC14, U4 OPA1678, U40 74HC14, U42 74HC237, U6 TMUX4053, U7 OPA1678, U8 LM3900, U9 OPA1679

Commit message: v2 proto passes DRC
Parts:
- removed J29: Conn_02x02_Odd_Even, Connector_PinHeader_2.54mm:PinHeader_2x02_P2.54mm_Vertical, symbol Connector_Generic:Conn_02x02_Odd_Even
- added J29, J34, J35, J43, J46, J47, J55, J56, J57, J58, J59, J61: GND, Connector_PinHeader_2.54mm:PinHeader_1x01_P2.54mm_Vertical, symbol Connector:Conn_01x01_Pin
- added J33: BOUNDS, Connector_PinHeader_2.00mm:PinHeader_1x01_P2.00mm_Vertical, symbol Connector:Conn_01x01_Pin
- added J45: SPARE_OUT, Connector_PinHeader_2.54mm:PinHeader_1x01_P2.54mm_Vertical, symbol Connector:Conn_01x01_Pin
- added J48, J52: +12V, Connector_PinHeader_2.54mm:PinHeader_1x01_P2.54mm_Vertical, symbol Connector:Conn_01x01_Pin
- added J49, J53: -12V, Connector_PinHeader_2.54mm:PinHeader_1x01_P2.54mm_Vertical, symbol Connector:Conn_01x01_Pin
- added J51, J54: +5V, Connector_PinHeader_2.54mm:PinHeader_1x01_P2.54mm_Vertical, symbol Connector:Conn_01x01_Pin
- added J62: INTEGRATOR_BUFFER, Connector_PinHeader_2.54mm:PinHeader_1x01_P2.54mm_Vertical, symbol Connector:Conn_01x01_Pin
- added J63: BIT1, Connector_PinHeader_2.54mm:PinHeader_1x01_P2.54mm_Vertical, symbol Connector:Conn_01x01_Pin
- added J66: BIT0, Connector_PinHeader_2.54mm:PinHeader_1x01_P2.54mm_Vertical, symbol Connector:Conn_01x01_Pin
- added J67: ENABLE_DECAY, Connector_PinHeader_2.54mm:PinHeader_1x01_P2.54mm_Vertical, symbol Connector:Conn_01x01_Pin
- added J68: AT_TARGET, Connector_PinHeader_2.00mm:PinHeader_1x01_P2.00mm_Vertical, symbol Connector:Conn_01x01_Pin
- added J69: EOA, Connector_PinHeader_2.54mm:PinHeader_1x01_P2.54mm_Vertical, symbol Connector:Conn_01x01_Pin
- added J70: DECAY_TRIG, Connector_PinHeader_2.54mm:PinHeader_1x01_P2.54mm_Vertical, symbol Connector:Conn_01x01_Pin
- added J71: DIR_CHANGE, Connector_PinHeader_2.54mm:PinHeader_1x01_P2.54mm_Vertical, symbol Connector:Conn_01x01_Pin
- added J72: MOVEMENT_TRIG, Connector_PinHeader_2.54mm:PinHeader_1x01_P2.54mm_Vertical, symbol Connector:Conn_01x01_Pin
- added J73: FILTERED_TRIG, Connector_PinHeader_2.54mm:PinHeader_1x01_P2.54mm_Vertical, symbol Connector:Conn_01x01_Pin
- added J74: FILTER_CRITERIA, Connector_PinHeader_2.54mm:PinHeader_1x01_P2.54mm_Vertical, symbol Connector:Conn_01x01_Pin
- J60: value Conn_01x02 -> SPARE_IN
Connections:
- net +12V: now also J48.1 (Pin_1), J52.1 (Pin_1)
- net +5V: now also J51.1 (Pin_1), J54.1 (Pin_1)
- net -12V: now also J49.1 (Pin_1), J53.1 (Pin_1)
- net AT_TARGET: now also J68.1 (Pin_1)
- net BIT0: now also J66.1 (Pin_1)
- net BIT1: now also J63.1 (Pin_1)
- net DECAY_TRIG: now also J70.1 (Pin_1)
- net DIRECTION: now also U39.5
- net DIR_CHANGE: now also J71.1 (Pin_1)
- net ENABLE_DECAY: now also J67.1 (Pin_1)
- net EOA: now also J69.1 (Pin_1)
- net FILTERED_TRIG: now also J73.1 (Pin_1)
- net FILTER_CRITERIA: now also J74.1 (Pin_1)
- net GND: now also J60.2 (Pin_2), J29.1 (Pin_1), J34.1 (Pin_1), J35.1 (Pin_1), J43.1 (Pin_1), J46.1 (Pin_1), J47.1 (Pin_1), J55.1 (Pin_1), J56.1 (Pin_1), J57.1 (Pin_1), J58.1 (Pin_1), J59.1 (Pin_1), J61.1 (Pin_1)
- net INV_DIRECTION: now also U39.6
- net MOVEMENT_TRIG: now also J72.1 (Pin_1)
- net ~{BOUNDS}: now also J33.1 (Pin_1)
- net at R82.2, R85.2, U33.1: now also J62.1 (Pin_1)
- net at U39.9: now also J60.1 (Pin_1)
- net at U39.8: now also J45.1 (Pin_1); no longer J60.2 (Pin_2)
Other:
- note added: "HOLD IN"
- moved on the sheet: J60, U39C

Commit message: update servo integrator to provide additional configuration options and add missing decoupling caps
Parts:
- added C63: DNP, Capacitor_SMD:C_0805_2012Metric, symbol Device:C
- added C64: 100n, Capacitor_SMD:C_0805_2012Metric, symbol Device:C_Small
- added D1, D2: 1N5819, Diode_SMD:D_SOD-123, symbol Device:D
- added J75: TRANSIMPEDANCE_AMP_OUT, Connector_PinHeader_2.54mm:PinHeader_1x01_P2.54mm_Vertical, symbol Connector:Conn_01x01_Pin
- added R72, R73: 10k, Resistor_SMD:R_0805_2012Metric, symbol Device:R
- added R74: 0R, Resistor_SMD:R_0805_2012Metric, symbol Device:R
- C48, C49, C56, C57: footprint (none) -> Capacitor_SMD:C_0805_2012Metric
- R88, R89: footprint (none) -> Resistor_SMD:R_0805_2012Metric
Connections:
- net GND: now also D1.2 (A), D2.1 (K)
- net INTEGRATOR_II_OUT: now also R73.2; no longer U35.6 (-)
- net at IC1.4 (OUT), R90.2, U33.6 (-): now also C63.1
- net at U35.2 (-), U6.14: now also R74.1; no longer C51.1
- net at R89.2, R90.1, U33.7: now also C63.2, J75.1 (Pin_1)
- net at U35.7, U6.13: now also C64.2, D1.1 (K), D2.2 (A), R72.2
- new net: C64.1, R72.1, R73.1, U35.6 (-)
- new net: C51.1, R74.2
Other:
- note added: "10-100 ohms for adjusting stability will introduce negligible HF error"
- note added: "Clamping diodes: keeps integrator close to GND when open-loop. Could be schottkys?"
- note added: "Consider reducing impedance to 7.5k"
- note added: "FILTER"
- moved on the sheet: C51

Commit message: update schematic with Will's debugging notes
Parts:
- added C14: C, symbol Device:C
- added C29: 100n, Capacitor_SMD:C_0805_2012Metric, symbol Device:C_Small
- added C36: 1200p, Capacitor_SMD:C_0805_2012Metric, symbol Device:C_Small
- added C65: DNP, Capacitor_SMD:C_0805_2012Metric, symbol Device:C
- added C68: 1.2n, Capacitor_SMD:C_0805_2012Metric, symbol Device:C
- added D10, D9: D, symbol Device:D
- added IC3: SSI2164, Package_SO:SOIC-16_3.9x9.9mm_P1.27mm, symbol custom_ic:SSI2164
- added J76: Conn_01x02, Connector_PinHeader_2.54mm:PinHeader_1x02_P2.54mm_Vertical, symbol Connector_Generic:Conn_01x02
- added J77: TRANSIMPEDANCE_AMP_OUT, Connector_PinHeader_2.54mm:PinHeader_1x01_P2.54mm_Vertical, symbol Connector:Conn_01x01_Pin
- added J78: INTEGRATOR_BUFFER, Connector_PinHeader_2.54mm:PinHeader_1x01_P2.54mm_Vertical, symbol Connector:Conn_01x01_Pin
- added R11: R, symbol Device:R
- added R12: 10k, Resistor_SMD:R_0805_2012Metric, symbol Device:R
- added R13, R14, R16, R17: 33k, Resistor_SMD:R_0805_2012Metric, symbol Device:R
- added R15: 220, Resistor_SMD:R_0805_2012Metric, symbol Device:R
- added R23, R27: 1M, Resistor_SMD:R_0805_2012Metric, symbol Device:R
- added R28, R29: 200k, Resistor_SMD:R_0805_2012Metric, symbol Device:R
- added U15: 74LS08, Package_SO:SOIC-14_3.9x8.7mm_P1.27mm, symbol 74xx:74LS08
- added U20: TLV1871, Package_TO_SOT_SMD:SOT-23-8, symbol Starling_Custom_IC:TLV1871
- added U21: 74HC74, Package_SO:SOIC-14_3.9x8.7mm_P1.27mm, symbol 74xx:74HC74
- added U23, U5: 74HC14, Package_SO:SOIC-14_3.9x8.7mm_P1.27mm, symbol 74xx:74HC14
- added U24, U27, U28: OPA1678, Package_SO:SOIC-8_3.9x4.9mm_P1.27mm, symbol Amplifier_Operational:OPA1678
- added U26: TMUX4053, Package_SO:TSSOP-16_4.4x5mm_P0.65mm, symbol custom_ic:TMUX4053
- added unit 4 of U6
Connections:
- net +12V: now also C29.1, R13.2, U20.8 (V+IN), U6.16 (VDD)
- net +5V: now also U20.6 (V+OUT), U21.2 (D), U21.4 (~{S})
- net -12V: now also U20.4 (V-IN)
- net ACTIVATION_TRIG: now also U5.5; no longer U1.1 (~{R})
- net AT_TARGET: now also J76.2 (Pin_2), U15.1; no longer U10.10, U10.2
- net GND: now also C14.2, C29.2, C36.1, C68.1, R12.1, R23.2, U20.1 (V-OUT), U24.5 (+), U6.6 (~{EN}), U6.7 (VEE), U6.8 (VSS); no longer U32.10 (T)
- net HOLD_REF: now also R14.1, U27.3 (+)
- net S+H_INTEGRATOR_OUT: now also R17.2, U28.1, U28.2 (-)
- net SLEW_CV: now also IC3.3 (CTRL)
- net ~{BOUNDS}: now also U15.2, U23.5
- new net: R27.1, R29.1, U24.2 (-)
- new net: C65.2, J77.1 (Pin_1), R16.1, R27.2, U24.7
- new net: C14.1, R11.2, U21.1 (~{R})
- new net: U21.3 (C), U23.6
- new net: R11.1, U21.6 (~{Q})
- new net: C65.1, IC3.4 (OUT), R16.2, U24.6 (-)
- new net: U5.2, U5.3
- new net: C68.2, R23.1, R28.1, U24.3 (+), U26.14, U28.3 (+)
- new net: J78.1 (Pin_1), R28.2, R29.2, U24.1
- new net: IC3.2 (IN), R14.2, R15.2
- new net: J76.1 (Pin_1), U26.11
- new net: D10.1 (K), D9.2 (A), R17.1, U27.2 (-)
- new net: D10.2 (A), D9.1 (K), U26.12, U27.1
- new net: U1.1 (~{R}), U5.6
- new net: C36.2, R15.1
- new net: R12.2, R13.1, U32.10 (T)
- new net BOUNDS_PULSE: U10.10, U10.2, U15.3
- new net OUTPUT_PULSE: U21.5 (Q)
Other:
- note added: "Do I need the two buffers?! Just feedback from the lower"
- note added: "Why 33k/30k? Limit clamp current?"
- moved on the sheet: C48, C49, J65
